File: pcb/stm32-40.sch (EAGLE design)
At the start: 63 parts, among them IC1 STM32F103RBT6, IC2 CAT24M01WI-GT3, IC3 AMIS30663CANG2G, IC4 MAX487-S, Q1 32768Hz, Q2 8MHz, SW1 KSS-2EG4430, X1 MCV3, X2 MCV3

Commit message: ...
Parts:
- added G1: (no value), battery:LI3VHOLDER
Connections:
- net GND: now also G1.-
- net VBAT: now also G1.+
Changed lines of the file:
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@@
 <grid distance="0.1" unitdist="inch" unit="inch" style="lines" multiple="1" display="no" altdistance="0.01" altunitdist="inch" altunit="inch"/>
 <layers>
-<layer number="1" name="Top" color="4" fill="1" visible="yes" active="no"/>
-<layer number="2" name="Route2" color="1" fill="3" visible="yes" active="no"/>
-<layer number="3" name="Route3" color="4" fill="3" visible="yes" active="no"/>
-<layer number="14" name="Route14" color="1" fill="6" visible="yes" active="no"/>
-<layer number="15" name="Route15" color="4" fill="6" visible="yes" active="no"/>
-<layer number="16" name="Bottom" color="1" fill="1" visible="yes" active="no"/>
-<layer number="17" name="Pads" color="2" fill="1" visible="yes" active="no"/>
-<layer number="18" name="Vias" color="2" fill="1" visible="yes" active="no"/>
-<layer number="19" name="Unrouted" color="6" fill="1" visible="yes" active="no"/>
-<layer number="20" name="Dimension" color="15" fill="1" visible="yes" active="no"/>
-<layer number="21" name="tPlace" color="7" fill="1" visible="yes" active="no"/>
-<layer number="22" name="bPlace" color="7" fill="1" visible="yes" active="no"/>
-<layer number="23" name="tOrigins" color="15" fill="1" visible="yes" active="no"/>
-<layer number="24" name="bOrigins" color="15" fill="1" visible="yes" active="no"/>
-<layer number="25" name="tNames" color="7" fill="1" visible="yes" active="no"/>
-<layer number="26" name="bNames" color="7" fill="1" visible="yes" active="no"/>
-<layer number="27" name="tValues" color="7" fill="1" visible="yes" active="no"/>
-<layer number="28" name="bValues" color="7" fill="1" visible="yes" active="no"/>
+<layer number="1" name="Top" color="4" fill="1" visible="no" active="no"/>
+<layer number="2" name="Route2" color="1" fill="3" visible="no" active="no"/>
+<layer number="3" name="Route3" color="4" fill="3" visible="no" active="no"/>
+<layer number="14" name="Route14" color="1" fill="6" visible="no" active="no"/>
+<layer number="15" name="Route15" color="4" fill="6" visible="no" active="no"/>
+<layer number="16" name="Bottom" color="1" fill="1" visible="no" active="no"/>
+<layer number="17" name="Pads" color="2" fill="1" visible="no" active="no"/>
+<layer number="18" name="Vias" color="2" fill="1" visible="no" active="no"/>
+<layer number="19" name="Unrouted" color="6" fill="1" visible="no" active="no"/>
+<layer number="20" name="Dimension" color="15" fill="1" visible="no" active="no"/>
+<layer number="21" name="tPlace" color="7" fill="1" visible="no" active="no"/>
+<layer number="22" name="bPlace" color="7" fill="1" visible="no" active="no"/>
+<layer number="23" name="tOrigins" color="15" fill="1" visible="no" active="no"/>
+<layer number="24" name="bOrigins" color="15" fill="1" visible="no" active="no"/>
+<layer number="25" name="tNames" color="7" fill="1" visible="no" active="no"/>
+<layer number="26" name="bNames" color="7" fill="1" visible="no" active="no"/>
+<layer number="27" name="tValues" color="7" fill="1" visible="no" active="no"/>
+<layer number="28" name="bValues" color="7" fill="1" visible="no" active="no"/>
 <layer number="29" name="tStop" color="7" fill="3" visible="no" active="no"/>
 <layer number="30" name="bStop" color="7" fill="6" visible="no" active="no"/>
@@
 <layer number="35" name="tGlue" color="7" fill="4" visible="no" active="no"/>
 <layer number="36" name="bGlue" color="7" fill="5" visible="no" active="no"/>
-<layer number="37" name="tTest" color="7" fill="1" visible="yes" active="no"/>
-<layer number="38" name="bTest" color="7" fill="1" visible="yes" active="no"/>
+<layer number="37" name="tTest" color="7" fill="1" visible="no" active="no"/>
+<layer number="38" name="bTest" color="7" fill="1" visible="no" active="no"/>
 <layer number="39" name="tKeepout" color="4" fill="11" visible="no" active="no"/>
 <layer number="40" name="bKeepout" color="1" fill="11" visible="no" active="no"/>
@@
 <layer number="44" name="Drills" color="7" fill="1" visible="no" active="no"/>
 <layer number="45" name="Holes" color="7" fill="1" visible="no" active="no"/>
-<layer number="46" name="Milling" color="3" fill="1" visible="yes" active="no"/>
-<layer number="47" name="Measures" color="7" fill="1" visible="yes" active="no"/>
-<layer number="48" name="Document" color="7" fill="1" visible="yes" active="no"/>
-<layer number="49" name="Reference" color="7" fill="1" visible="yes" active="no"/>
-<layer number="50" name="dxf" color="7" fill="1" visible="yes" active="no"/>
-<layer number="51" name="tDocu" color="7" fill="1" visible="yes" active="no"/>
-<layer number="52" name="bDocu" color="7" fill="1" visible="yes" active="no"/>
-<layer number="53" name="tGND_GNDA" color="7" fill="9" visible="yes" active="no"/>
-<layer number="54" name="bGND_GNDA" color="1" fill="9" visible="yes" active="no"/>
-<layer number="56" name="wert" color="7" fill="1" visible="yes" active="no"/>
+<layer number="46" name="Milling" color="3" fill="1" visible="no" active="no"/>
+<layer number="47" name="Measures" color="7" fill="1" visible="no" active="no"/>
+<layer number="48" name="Document" color="7" fill="1" visible="no" active="no"/>
+<layer number="49" name="Reference" color="7" fill="1" visible="no" active="no"/>
+<layer number="50" name="dxf" color="7" fill="1" visible="no" active="no"/>
+<layer number="51" name="tDocu" color="7" fill="1" visible="no" active="no"/>
+<layer number="52" name="bDocu" color="7" fill="1" visible="no" active="no"/>
+<layer number="53" name="tGND_GNDA" color="7" fill="9" visible="no" active="no"/>
+<layer number="54" name="bGND_GNDA" color="1" fill="9" visible="no" active="no"/>
+<layer number="56" name="wert" color="7" fill="1" visible="no" active="no"/>
 <layer number="91" name="Nets" color="2" fill="1" visible="yes" active="yes"/>
 <layer number="92" name="Busses" color="1" fill="1" visible="yes" active="yes"/>
@@
 <part name="X2" library="con-phoenix-381_l" deviceset="MCV3" device=""/>
 <part name="GND8" library="rs485" deviceset="GND" device=""/>
+<part name="G1" library="battery" deviceset="LI3VHOLDER" device=""/>
+<part name="GND9" library="rs485" deviceset="GND" device=""/>
 </parts>
 <sheets>
@@
 <attribute name="VALUE" x="85.979" y="132.588" size="1.778" layer="96" rot="R90"/>
 </instance>
+<instance part="G1" gate="G$1" x="144.78" y="149.86" rot="R90"/>
+<instance part="GND9" gate="1" x="144.78" y="142.24"/>
 </instances>
 <busses>
@@
 <pinref part="C17" gate="G$1" pin="2"/>
 </segment>
+<segment>
+<pinref part="G1" gate="G$1" pin="-"/>
+<pinref part="GND9" gate="1" pin="GND"/>
+</segment>
 </net>
 <net name="BOOT1" class="0">
@@
 <segment>
 <wire x1="193.04" y1="160.02" x2="187.96" y2="160.02" width="0.1524" layer="91"/>
-<wire x1="187.96" y1="160.02" x2="177.8" y2="160.02" width="0.1524" layer="91"/>
+<wire x1="187.96" y1="160.02" x2="144.78" y2="160.02" width="0.1524" layer="91"/>
+<wire x1="144.78" y1="160.02" x2="139.7" y2="160.02" width="0.1524" layer="91"/>
 <wire x1="187.96" y1="157.48" x2="187.96" y2="160.02" width="0.1524" layer="91"/>
 <junction x="187.96" y="160.02"/>
-<label x="177.8" y="160.02" size="1.778" layer="95" rot="R180" xref="yes"/>
+<label x="139.7" y="160.02" size="1.778" layer="95" rot="R180" xref="yes"/>
 <pinref part="IC1" gate="G$1" pin="VBAT"/>
 <pinref part="C15" gate="G$1" pin="1"/>
-</segment>
-</net>
+<pinref part="G1" gate="G$1" pin="+"/>
+<wire x1="144.78" y1="154.94" x2="144.78" y2="160.02" width="0.1524" layer="91"/>
+<junction x="144.78" y="160.02"/>
+</segment>
+</net>

Commit message: ...
Parts:
- removed C15: 0.1, rc-master-smd:C_0603
- added JP2: (no value), stamp:UART-5_2.54
- added R9: 10K, rc-master-smd:R_0603
Connections:
- removed net PC10: IC1.PC10/(USART3_TX)
- removed net PC11: IC1.PC11/(USART3_RX)
- removed net PC12: IC1.PC12/(USART3_CK)
- removed net U3_DE: IC4G$1.DE, IC4G$1.RE/, R7.2
- removed net U3_RX: IC4G$1.RO
- removed net U3_TX: IC4G$1.DI
- new net DE3: IC1.PC12/(USART3_CK), IC4G$1.DI
- new net RXD3: IC1.PC11/(USART3_RX), IC4G$1.RO
- new net TXD3: IC1.PC10/(USART3_TX), IC4G$1.DE, IC4G$1.RE/, R7.2
- net +3V3: now also R9.2
- net GND: now also JP2.1; no longer C15.2
- net RXD1: now also JP2.3, R9.1
- net TXD1: now also JP2.2
- net VBAT: no longer C15.1

Commit message: route timers
Parts:
- removed R17: 330, rc-master-smd:R_0603
- added C15: 0.1, rc-master-smd:C_0805
- added C18, C19: 100uF/6V3, rc-master-smd:CP_SMCD
- added R10, R11, R12, R22, R23, R24, R25, R26, R27, R28, R29, R30: 10, rc-master-smd:R_0603
- added U1: (no value), vreg-linear:LM1117-3.3
- C14: device rc-master-smd:C_0603 -> rc-master-smd:C_0805
- Q1: device discrete:CRYSTAL-TC26H -> discrete:CRYSTAL-TC38H
Connections:
- removed net N$11: R17.2
- removed net N$14: R8.1
- new net N$15: R10.1, STMP1G$1.2
- new net N$16: R11.1, STMP1G$1.3
- new net N$17: R12.1, STMP1G$1.4
- new net N$18: R22.1, STMP1G$1.5
- new net N$19: R23.1, STMP1G$1.7
- new net N$20: R24.1, STMP1G$1.8
- new net N$21: R25.1, STMP1G$1.9
- new net N$22: R26.1, STMP1G$1.10
- new net N$23: R27.1, STMP1G$1.12
- new net N$24: R28.1, STMP1G$1.13
- new net N$25: R29.1, STMP1G$1.14
- new net N$26: R30.1, STMP1G$1.15
- net +3V3: now also C15.1, C19.+, U1.OUT; no longer C14.1
- net +5V: now also C14.1, C18.+, STMP1G$1.20, U1.IN
- net GND: now also C15.2, C18.-, C19.-, STMP1G$1.1, STMP1G$1.11, STMP1G$1.19, STMP1G$1.6, U1.GND; no longer S1.2
- net N$8: now also R8.2; no longer R17.1
- net PC0: now also R27.2
- net PC1: now also R28.2
- net PC2: now also R29.2
- net PC3: now also R30.2
- net RS485_A: now also R8.1; no longer R8.2
- net RS485_B: now also S1.2
- net TIM3_CH1: now also R10.2
- net TIM3_CH2: now also R11.2
- net TIM3_CH3: now also R12.2
- net TIM3_CH4: now also R22.2
- net TIM4_CH1: now also R23.2
- net TIM4_CH2: now also R24.2
- net TIM4_CH3: now also R25.2
- net TIM4_CH4: now also R26.2
Other:
- moved on the sheet: C14, C16, R8, STMP1G$1, STMP1G$2

Commit message: route in progress
Parts:
- removed JP1: (no value), pinhead-fixdrills:PINHD-1X2_2.54
- added R34, R37: 560, rc-master-smd:R_0603
- added SW2: KSS-2EG4430, buttons:KSS-2EG4430
- Q1: device discrete:CRYSTAL-TC38H -> crystal:CRSTL3-
Connections:
- removed net N$12: R18.2
- removed net N$13: R19.2
- removed net N$25: R29.1, STMP1G$1.14
- removed net N$26: R30.1, STMP1G$1.15
- removed net PB5: IC1.PB5/I2C1_SMBA/(TIM3_CH2/SPI1_MOSI)
- new net N$11: R27.1, STMP1G$1.11
- new net N$14: R28.1, STMP1G$1.12
- new net SW3: IC1.JTDO/(TIM2_CH2/PB3/TRACESWO/SPI1_SCK), R18.2
- new net SW4: IC1.JTNRST/(PB4/TIM3_CH1/SPI1_MISO), R19.2
- net +3V3: now also JP2.5, SW2.S; no longer JP1.1
- net +5V: now also JP2.4, R34.2
- net BOOT0: now also IC1.PB5/I2C1_SMBA/(TIM3_CH2/SPI1_MOSI)
- net GND: now also Q1.P$1, R37.1, STMP1G$1.10; no longer STMP1G$1.11, STMP1G$1.6
- net N$19: now also STMP1G$1.6; no longer STMP1G$1.7
- net N$20: now also STMP1G$1.7; no longer STMP1G$1.8
- net N$21: now also STMP1G$1.8; no longer STMP1G$1.9
- net N$22: now also STMP1G$1.9; no longer STMP1G$1.10
- net N$23: now also R29.1, STMP1G$1.13; no longer R27.1, STMP1G$1.12
- net N$24: now also R30.1, STMP1G$1.14; no longer R28.1, STMP1G$1.13
- net N$3: now also SW2.P; no longer JP1.2
- net N$44: now also R34.1
- net N$6: now also R37.2
Other:
- moved on the sheet: C13, C21, C22, C24, C25, D1, D2, F1, F2, F3, F4, IC3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

Commit message: pcb in progress
Parts:
- removed C13: 0.1, rc-master-smd:C_0603
- removed C24: 560pF, rc-master-smd:C_0603
- removed R37: 560, rc-master-smd:R_0603
- removed R38: NC, rc-master-smd:R_0603
- added C20: 0.1, rc-master-smd:C_0603
- added LED2: (no value), led:LEDCHIP-LED0805
- added R17: 10, rc-master-smd:R_0603
- added R31: 330, rc-master-smd:R_0603
- added R33: 100, rc-master-smd:R_0603
- C14: value 0.1 -> 100uF/6V3; device rc-master-smd:C_0805 -> rc-master-smd:CP_SMCD
- C16: value 0.1 -> 100uF/6V3; device rc-master-smd:C_0603 -> rc-master-smd:CP_SMCD
- C17: device rc-master-smd:C_0603 -> rc-master-smd:C_0805
- C18, C19: value 100uF/6V3 -> 0.1; device rc-master-smd:CP_SMCD -> rc-master-smd:C_0603
- C22: value 0.1 -> 560pF
- IC3: value AMIS30663CANG2G -> MAX487-S; device interfaces:SN65HVD230 -> rs232-rs485:MAX487-S
- IC4: value MAX487-S -> AMIS30663CANG2G; device rs232-rs485:MAX487-S -> interfaces:SN65HVD230
- R10, R26: value 10 -> 10K
- R11, R12: value 10 -> 4.7K
- R13, R14: value 4.7K -> 10
- R15: value 100 -> 10
- R16: value 120 -> 10; device rc-master-smd:R_0805 -> rc-master-smd:R_0603
- R18, R19: value 330 -> 10
- R2: value 10K -> 220
- R20, R21: value 10K -> 10
- R25, R27: value 10 -> 560
- R28, R30: value 10 -> 120; device rc-master-smd:R_0603 -> rc-master-smd:R_0805
- R29: value 10 -> 330
- R34: value 560 -> 100
- R36: value 100 -> NC
- R4: value 2.2K -> 10K
- R5: value 1M -> 10K
- R6: value 10K -> 2.2K
- R7: value 10K -> 1M
- R8: value 120 -> 10K; device rc-master-smd:R_0805 -> rc-master-smd:R_0603
- renumbered C25 to C23, JP4 to JP1
Connections:
- new net N$30: LED2.A, R2.2
- net !RESET: now also R8.1, SW2.S; no longer R6.1, SW1.S
- net +3V3: now also C16.+, C20.1, C7.1, R1.1, R10.2, R11.2, R12.2, R5.2, R8.2, SW1.S; no longer C17.1, C19.+, C22.1, R13.2, R14.2, R20.2, R21.2, R6.2, SW2.S
- net +5V: now also C14.+, C17.1, C18.1, C19.1, IC3G$2.VCC, IC4.VDD, R25.2; no longer C14.1, C18.+, C21.1, C7.1, IC3.VDD, IC4G$2.VCC, R34.2
- net BOOT0: now also R4.1; no longer R3.1
- net BOOT1: now also R3.1; no longer R1.1
- net CAN_CTRL: now also IC4.RS, R36.2; no longer IC3.RS, R38.2
- net CAN_H: now also F3.2, R30.1, X2.1.SK; no longer F2.2, R16.1, X1.1.SK
- net CAN_L: now also F4.2, X2.3.SK; no longer F3.2, X1.3.SK
- net CAN_RX: now also R33.1; no longer R15.1
- net CAN_TX: now also IC4.TXD; no longer IC3.TXD
- net DE3: now also IC3G$1.DI; no longer IC4G$1.DI
- net GND: now also C14.-, C16.-, C18.2, C19.2, C20.2, IC3G$2.GND, IC4.VSS, LED2.C, R26.1, R27.1, R3.2, R36.1, R6.1, STMP1G$2.1, STMP1G$2.20, SW2.P; no longer C13.2, C14.2, C16.2, C18.-, C19.-, C24.2, IC3.VSS, IC4G$2.GND, R2.2, R37.1, R38.1, R4.1, R7.1, SW1.P
- net N$1: now also C21.1, IC4.VREF; no longer C13.1, IC3.VREF
- net N$10: now also R31.1; no longer R19.1
- net N$11: now also R21.1; no longer R27.1
- net N$14: now also R22.1; no longer R28.1
- net N$15: now also R13.1; no longer R10.1
- net N$16: now also R14.1; no longer R11.1
- net N$17: now also R15.1; no longer R12.1
- net N$18: now also R16.1; no longer R22.1
- net N$19: now also R17.1; no longer R23.1
- net N$2: now also R30.2; no longer R16.2
- net N$20: now also R18.1; no longer R24.1
- net N$21: now also R19.1; no longer R25.1
- net N$22: now also R20.1; no longer R26.1
- net N$23: now also R23.1; no longer R29.1
- net N$24: now also R24.1; no longer R30.1
- net N$3: now also R6.2, SW1.P; no longer R3.2, SW2.P
- net N$44: now also F2.1, IC3G$1.A, R25.1; no longer F4.1, IC4G$1.A, R34.1
- net N$51: now also F3.1, IC4.CANH, R34.2; no longer F2.1, IC3.CANH, R35.2
- net N$52: now also F4.1, IC4.CANL, R35.2; no longer F3.1, IC3.CANL, R36.2
- net N$54: now also R35.1; no longer R36.1
- net N$55: now also C22.1, R34.1; no longer C24.1, R35.1
- net N$6: now also IC3G$1.B, R27.2; no longer IC4G$1.B, R37.2
- net N$7: now also IC4.RXD, R33.2; no longer IC3.RXD, R15.2
- net N$8: now also R28.2; no longer R8.2
- net N$9: now also R29.1; no longer R18.1
- net OSC_IN: now also R7.2; no longer R5.2
- net OSC_OUT: now also R7.1; no longer R5.1
- net PC0: now also R21.2; no longer R27.2
- net PC1: now also R22.2; no longer R28.2
- net PC13: now also STMP1G$2.19
- net PC2: now also R23.2; no longer R29.2
- net PC3: now also R24.2; no longer R30.2
- net RS485_A: now also F2.2, R28.1, X1.1.SK; no longer F4.2, R8.1, X2.1.SK
- net RS485_B: now also X1.3.SK; no longer X2.3.SK
- net RXD1: now also R5.1; no longer R9.1
- net RXD3: now also IC3G$1.RO; no longer IC4G$1.RO
- net SCL2: now also R11.1; no longer R13.1
- net SDA2: now also R12.1; no longer R14.1
- net SW3: now also R29.2; no longer R18.2
- net SW4: now also R31.2; no longer R19.2
- net SWCLK: now also R9.1; no longer R20.1
- net SWDIO: now also R10.1; no longer R21.1
- net TIM3_CH1: now also R13.2; no longer R10.2
- net TIM3_CH2: now also R14.2; no longer R11.2
- net TIM3_CH3: now also R15.2; no longer R12.2
- net TIM3_CH4: now also R16.2; no longer R22.2
- net TIM4_CH1: now also R17.2; no longer R23.2
- net TIM4_CH2: now also R18.2; no longer R24.2
- net TIM4_CH3: now also R19.2; no longer R25.2
- net TIM4_CH4: now also R20.2; no longer R26.2
- net TXD3: now also IC3G$1.DE, IC3G$1.RE/, R26.2; no longer IC4G$1.DE, IC4G$1.RE/, R7.2
- net VDDA: no longer C16.1
Other:
- note added: "Power LED"
- moved on the sheet: C21, C22, F2, F3, F4, LED1, R1, R2, R27, R3, R34, R35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

Commit message: pcb in progress
Connections:
- net PA0: now also STMP1G$2.2
- net PA1: now also STMP1G$2.3
- net PA2: now also STMP1G$2.4
- net PA3: now also STMP1G$2.5
- net PA4: now also STMP1G$2.6
- net PA5: now also STMP1G$2.7
- net PA6: now also STMP1G$2.8
- net PA7: now also STMP1G$2.9
Changed lines of the file:
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@@
+</segment>
+</net>
+<net name="PA0" class="0">
+<segment>
+<pinref part="STMP1" gate="G$2" pin="2"/>
+<wire x1="132.08" y1="226.06" x2="106.68" y2="226.06" width="0.1524" layer="91"/>
+<label x="109.22" y="226.06" size="1.778" layer="95"/>
+</segment>
+</net>
+<net name="PA1" class="0">
+<segment>
+<pinref part="STMP1" gate="G$2" pin="3"/>
+<wire x1="106.68" y1="223.52" x2="132.08" y2="223.52" width="0.1524" layer="91"/>
+<label x="109.22" y="223.52" size="1.778" layer="95"/>
+</segment>
+</net>
+<net name="PA2" class="0">
+<segment>
+<pinref part="STMP1" gate="G$2" pin="4"/>
+<wire x1="132.08" y1="220.98" x2="106.68" y2="220.98" width="0.1524" layer="91"/>
+<label x="109.22" y="220.98" size="1.778" layer="95"/>
+</segment>
+</net>
+<net name="PA3" class="0">
+<segment>
+<pinref part="STMP1" gate="G$2" pin="5"/>
+<wire x1="106.68" y1="218.44" x2="132.08" y2="218.44" width="0.1524" layer="91"/>
+<label x="109.22" y="218.44" size="1.778" layer="95"/>
+</segment>
+</net>
+<net name="PA4" class="0">
+<segment>
+<pinref part="STMP1" gate="G$2" pin="6"/>
+<wire x1="132.08" y1="215.9" x2="106.68" y2="215.9" width="0.1524" layer="91"/>
+<label x="109.22" y="215.9" size="1.778" layer="95"/>
+</segment>
+</net>
+<net name="PA5" class="0">
+<segment>
+<pinref part="STMP1" gate="G$2" pin="7"/>
+<wire x1="106.68" y1="213.36" x2="132.08" y2="213.36" width="0.1524" layer="91"/>
+<label x="109.22" y="213.36" size="1.778" layer="95"/>
+</segment>
+</net>
+<net name="PA6" class="0">
+<segment>
+<pinref part="STMP1" gate="G$2" pin="8"/>
+<wire x1="132.08" y1="210.82" x2="106.68" y2="210.82" width="0.1524" layer="91"/>
+<label x="109.22" y="210.82" size="1.778" layer="95"/>
+</segment>
+</net>
+<net name="PA7" class="0">
+<segment>
+<pinref part="STMP1" gate="G$2" pin="9"/>
+<wire x1="132.08" y1="208.28" x2="106.68" y2="208.28" width="0.1524" layer="91"/>
+<label x="109.22" y="208.28" size="1.778" layer="95"/>
 </segment>
 </net>
