File: pcb/stm32-dip40.brd (EAGLE design)
At the start: 57.1 x 17.8 mm, 32 parts, among them IC1 TODO AMIS30663CANG2G, IC2 STM32F103C8, J1 DIP-40, Q1 32768Hz, Q2 8MHz, X1 DG3XX-03-3.5

Commit message: dip40 in progress
Parts:
- Q1: device discrete:TC26H -> crystal:TC38H-G
- moved Q1 40.9 mm to (47.4, 13.0), turned to 180 degrees
- moved R1 40.8 mm to (47.4, 11.2), flipped to the bottom
- moved C2 39.4 mm to (48.2, 8.86), flipped to the bottom, turned to 270 degrees
- moved R2 29.9 mm to (39.5, 7.92), flipped to the bottom
- moved Q2 29.1 mm to (39.5, 7.98), turned to 180 degrees
- moved C3 28.7 mm to (42.4, 4.64), turned to 180 degrees
- moved C4 24.8 mm to (39.2, 4.66)
- moved C1 23.3 mm to (46.6, 8.84), flipped to the bottom, turned to 270 degrees
- moved R10 8.25 mm to (46.4, 14.8), turned to 180 degrees
- moved R9 8.10 mm to (49.6, 14.8), turned to 0 degrees
- moved L1 2.16 mm to (22.8, 14.0), turned to 225 degrees
- moved C8 0.71 mm to (28.7, 13.8)
Connections:
- removed net OSC_IN1: C3.1, IC2.5, Q2.1, R2.1
- removed net OSC_OUT1: C4.1, IC2.6, Q2.2, R2.2
- removed net PA10: IC2.31
- removed net PA9: IC2.30
- removed net PB10: J1.4
- removed net SWO: IC2.39, SWD1.6
- new net PB3/SWO: IC2.39, J1.4, SWD1.6
- new net PB4: IC2.40, J1.24
- new net PB5: IC2.41, J1.25
- new net RXD1: IC2.31, J1.14
- new net TXD1: IC2.30, J1.15
- net PA15: now also J1.21
- net PA8: now also J1.20
- net SWCLK: now also J1.19
- net SWDIO: now also J1.18
- net USBDM: now also J1.16
- net USBDP: now also J1.17
- net XTAL1: now also C3.1, IC2.5, Q2.1, R2.1
- net XTAL2: now also C4.1, IC2.6, Q2.2, R2.2
Routing:
- net PB3/SWO: track 0.00 -> 54.1 mm, vias 0 -> 4
- net XTAL1: track 0.00 -> 35.4 mm, vias 0 -> 1
- net XTAL2: track 0.00 -> 29.7 mm, vias 0 -> 1
- net OSC32_OUT: track 0.00 -> 27.6 mm, vias 0 -> 1
- net PA15: track 0.00 -> 25.6 mm
- net OSC32_IN: track 0.00 -> 25.1 mm, vias 0 -> 1
- net PA8: track 0.00 -> 24.1 mm, vias 0 -> 1
- net I2C1_SCL: track 0.00 -> 20.8 mm
- net I2C1_SDA: track 0.00 -> 20.0 mm
- net PB4: track 0.00 -> 17.5 mm, vias 0 -> 1
- net !RESET: track 0.00 -> 17.0 mm, vias 0 -> 1
- net PB5: track 0.00 -> 16.5 mm, vias 0 -> 1
- net USBDP: track 0.00 -> 14.9 mm
- net USBDM: track 0.00 -> 12.6 mm
- net SWDIO: track 27.9 -> 39.7 mm
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