File: pcb/stm32-dip40.sch (EAGLE design)
At the start: 32 parts, among them IC1 TODO AMIS30663CANG2G, IC2 STM32F103C8, J1 DIP-40, Q1 32768Hz, Q2 8MHz, X1 DG3XX-03-3.5

Commit message: dip40 in progress
Parts:
- Q1: device discrete:CRYSTAL-TC26H -> crystal:CRYSTAL-TC38H-G
Connections:
- removed net OSC_IN1: C3.1, IC2.OSC_IN/(PD0/CANRX), Q2.1, R2.1
- removed net OSC_OUT1: C4.1, IC2.OSC_OUT/(PD1/CANTX), Q2.2, R2.2
- removed net PA10: IC2.PA10/USART1_RX/TIM1_CH3
- removed net PA9: IC2.PA9/USART1_TX/TIM1_CH2
- removed net PB10: J1.1.4
- removed net SWO: IC2.JTDO/(TIM2_CH2/PB3/TRACESWO/SPI1_SCK), SWD1.6
- new net PB3/SWO: IC2.JTDO/(TIM2_CH2/PB3/TRACESWO/SPI1_SCK), J1.1.4, SWD1.6
- new net PB4: IC2.JTNRST/(PB4/TIM3_CH1/SPI1_MISO), J1.2.4
- new net PB5: IC2.PB5/I2C1_SMBA/(TIM3_CH2/SPI1_MOSI), J1.2.5
- new net RXD1: IC2.PA10/USART1_RX/TIM1_CH3, J1.1.14
- new net TXD1: IC2.PA9/USART1_TX/TIM1_CH2, J1.1.15
- net PA15: now also J1.2.1
- net PA8: now also J1.1.20
- net SWCLK: now also J1.1.19
- net SWDIO: now also J1.1.18
- net USBDM: now also J1.1.16
- net USBDP: now also J1.1.17
- net XTAL1: now also C3.1, IC2.OSC_IN/(PD0/CANRX), Q2.1, R2.1
- net XTAL2: now also C4.1, IC2.OSC_OUT/(PD1/CANTX), Q2.2, R2.2
