File: pcb/stm32-40.brd (EAGLE design)
At the start: 63.5 x 57.1 mm, 63 parts, among them IC1 STM32F103RBT6, IC2 CAT24M01WI-GT3, IC3 AMIS30663CANG2G, IC4 MAX487-S, Q1 32768Hz, Q2 8MHz, SW1 KSS-2EG4430, X1 MCV3, X2 MCV3

Commit message: ...
Parts:
- added G1: (no value), battery:LITHOLDER
Connections:
- net GND: now also G1.-
- net VBAT: now also G1.+
Routing:
- net SDA2: track 36.6 -> 0.00 mm, vias 2 -> 0
- net PC12: track 13.1 -> 0.00 mm, vias 1 -> 0
- net VBAT: track 12.6 -> 0.00 mm
- net PC10: track 12.4 -> 0.00 mm, vias 1 -> 0
- net PD2: track 12.3 -> 0.00 mm, vias 1 -> 0
- net PC11: track 12.1 -> 0.00 mm, vias 1 -> 0
- net PC13: track 10.9 -> 0.00 mm
Changed lines of the file:
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@@
 <attribute name="VALUE" x="12.954" y="20.32" size="1.778" layer="27" ratio="10" rot="R90"/>
 </element>
+<element name="G1" library="battery" package="LITHOLDER" value="" x="14.605" y="-15.24"/>
 </elements>
 <signals>
@@
 <contactref element="D1" pad="3"/>
 <contactref element="X2" pad="2"/>
+<contactref element="G1" pad="-"/>
 <wire x1="78.4225" y1="82.8675" x2="81.28" y2="82.7087" width="0" layer="19" extent="1-1"/>
 <wire x1="77.1525" y1="82.8675" x2="78.4225" y2="82.8675" width="0" layer="19" extent="1-1"/>
@@
 <wire x1="16.655" y1="66.675" x2="16.655" y2="64.135" width="0" layer="19" extent="1-1"/>
 <wire x1="16.655" y1="69.215" x2="16.655" y2="66.675" width="0" layer="19" extent="1-1"/>
+<wire x1="14.605" y1="-23.495" x2="22.352" y2="22.86" width="0" layer="19" extent="1-1"/>
 </signal>
 <signal name="BOOT1">
@@
 <contactref element="IC1" pad="1"/>
 <contactref element="C15" pad="1"/>
-<wire x1="52.72" y1="81.22" x2="52.13" y2="81.22" width="0.254" layer="1"/>
-<wire x1="52.13" y1="81.22" x2="52.07" y2="81.28" width="0.254" layer="1"/>
-<wire x1="52.07" y1="81.28" x2="52.07" y2="90.805" width="0.254" layer="1"/>
-<wire x1="50.9905" y1="91.8845" x2="50.9905" y2="92.71" width="0.254" layer="1"/>
-<wire x1="52.07" y1="90.805" x2="50.9905" y2="91.8845" width="0.254" layer="1"/>
+<contactref element="G1" pad="+"/>
+<wire x1="52.72" y1="81.22" x2="50.9905" y2="92.71" width="0" layer="19" extent="1-1"/>
+<wire x1="14.605" y1="-3.175" x2="52.72" y2="81.22" width="0" layer="19" extent="1-1"/>
 </signal>
 <signal name="N$30">
@@
 <signal name="PC13">
 <contactref element="IC1" pad="2"/>
-<wire x1="51.6775" y1="80.72" x2="52.72" y2="80.72" width="0.254" layer="1"/>
-<wire x1="51.435" y1="80.9625" x2="51.6775" y2="80.72" width="0.254" layer="1"/>
-<wire x1="51.435" y1="80.9625" x2="51.435" y2="90.4875" width="0.254" layer="1"/>
 </signal>
 <signal name="SPI2_NSS">
@@
 <signal name="PD2">
 <contactref element="IC1" pad="54"/>
-<wire x1="59.67" y1="83.17" x2="59.67" y2="88.0862" width="0.254" layer="1"/>
-<wire x1="59.67" y1="88.0862" x2="60.0075" y2="88.4237" width="0.254" layer="1"/>
-<wire x1="60.0075" y1="88.4237" x2="60.0075" y2="92.71" width="0.254" layer="16"/>
-<wire x1="60.0075" y1="92.71" x2="58.7375" y2="93.98" width="0.254" layer="16"/>
-<wire x1="58.7375" y1="93.98" x2="57.88" y2="93.98" width="0.254" layer="16"/>
-<via x="60.0075" y="88.4237" extent="1-16" drill="0.4"/>
 </signal>
 <signal name="+5V">
@@
 <contactref element="IC2" pad="5"/>
 <contactref element="R14" pad="1"/>
-<wire x1="37.7825" y1="69.5325" x2="37.7825" y2="71.628" width="0.3048" layer="1"/>
-<wire x1="61.17" y1="69.64" x2="61.17" y2="71.77" width="0.254" layer="1"/>
-<wire x1="61.9125" y1="68.8975" x2="61.17" y2="69.64" width="0.254" layer="1"/>
-<wire x1="61.7538" y1="68.8975" x2="61.9125" y2="68.8975" width="0.254" layer="1"/>
-<wire x1="61.7538" y1="68.8975" x2="62.0713" y2="68.1038" width="0.254" layer="1"/>
-<wire x1="62.0713" y1="68.1038" x2="61.9125" y2="67.6275" width="0.254" layer="1"/>
-<wire x1="39.6875" y1="68.8975" x2="61.7538" y2="68.8975" width="0.254" layer="16"/>
-<wire x1="38.735" y1="67.31" x2="38.735" y2="67.945" width="0.254" layer="16"/>
-<wire x1="38.735" y1="67.945" x2="39.6875" y2="68.8975" width="0.254" layer="16" curve="-89.987971"/>
-<wire x1="38.735" y1="67.31" x2="37.7825" y2="69.5325" width="0.254" layer="1" curve="-46.396648"/>
-<wire x1="41.8084" y1="66.04" x2="38.735" y2="67.31" width="0.254" layer="1" curve="-42.304145"/>
-<via x="61.7538" y="68.8975" extent="1-16" drill="0.4"/>
-<via x="38.735" y="67.31" extent="1-16" drill="0.4"/>
+<wire x1="41.8084" y1="66.04" x2="61.17" y2="71.77" width="0" layer="19" extent="1-1"/>
+<wire x1="37.7825" y1="71.628" x2="41.8084" y2="66.04" width="0" layer="19" extent="1-1"/>
 </signal>
 <signal name="PC12">
 <contactref element="IC1" pad="53"/>
-<wire x1="60.17" y1="83.17" x2="60.17" y2="87.475" width="0.254" layer="1"/>
-<wire x1="60.17" y1="87.475" x2="60.8013" y2="88.1062" width="0.254" layer="1"/>
-<wire x1="60.8013" y1="88.1062" x2="60.8013" y2="89.2176" width="0.254" layer="1"/>
-<wire x1="60.8013" y1="89.2176" x2="60.8013" y2="92.8687" width="0.254" layer="16"/>
-<wire x1="60.8013" y1="92.8687" x2="58.61" y2="95.06" width="0.254" layer="16"/>
-<via x="60.8013" y="89.2176" extent="1-16" drill="0.4"/>
 </signal>
 <signal name="PC11">
 <contactref element="IC1" pad="52"/>
-<wire x1="60.67" y1="83.17" x2="60.67" y2="87.1812" width="0.254" layer="1"/>
-<wire x1="60.67" y1="87.1812" x2="61.595" y2="88.1062" width="0.254" layer="1"/>
-<wire x1="61.595" y1="88.1062" x2="61.595" y2="90.0113" width="0.254" layer="1"/>
-<wire x1="61.595" y1="90.0113" x2="61.5951" y2="93.5039" width="0.254" layer="16"/>
-<wire x1="61.5951" y1="93.5039" x2="60.61" y2="94.4888" width="0.254" layer="16"/>
-<via x="61.595" y="90.0113" extent="1-16" drill="0.4"/>
 </signal>
 <signal name="PC10">
 <contactref element="IC1" pad="51"/>
-<wire x1="61.17" y1="83.17" x2="61.17" y2="86.8875" width="0.254" layer="1"/>
-<wire x1="61.17" y1="86.8875" x2="62.3888" y2="88.1062" width="0.254" layer="1"/>
-<wire x1="62.3888" y1="88.1062" x2="62.3888" y2="89.3762" width="0.254" layer="1"/>
-<wire x1="62.3888" y1="89.3762" x2="62.3887" y2="89.5351" width="0.254" layer="16"/>
-<wire x1="62.3887" y1="89.5351" x2="62.3887" y2="95.0288" width="0.254" layer="16"/>
-<via x="62.3888" y="89.3762" extent="1-16" drill="0.4"/>
 </signal>
 <signal name="TIM3_CH4">
@@
 <contactref element="R8" pad="2"/>
 <contactref element="X2" pad="1"/>
+<wire x1="13.39" y1="22.86" x2="7.62" y2="22.86" width="0.4064" layer="1"/>
 <wire x1="13.39" y1="22.86" x2="12.7" y2="25.654" width="0" layer="19" extent="1-1"/>
-<wire x1="13.39" y1="22.86" x2="7.62" y2="22.86" width="0.4064" layer="1"/>
 </signal>
 <signal name="N$44">

Commit message: ...
Parts:
- removed C15: 0.1, rc-master-smd:C0603
- added JP2: (no value), stamp:UART_1X05
- added R9: 10K, rc-master-smd:R0603
- moved C14 70.0 mm to (40.6, 24.1), turned to 180 degrees
- moved C4 63.6 mm to (54.3, 27.3), turned to 270 degrees
- moved C3 63.1 mm to (52.7, 27.3), turned to 270 degrees
- moved C2 62.5 mm to (50.5, 27.3), turned to 270 degrees
- moved C1 62.3 mm to (48.9, 27.3), turned to 270 degrees
- moved C10 55.4 mm to (31.1, 36.2), turned to 180 degrees
- moved C11 51.8 mm to (40.0, 33.7), turned to 90 degrees
- moved Q2 47.6 mm to (51.4, 34.9), turned to 90 degrees
- moved R5 47.6 mm to (51.4, 34.9), turned to 270 degrees
- moved Q1 45.2 mm to (46.4, 35.9), turned to 180 degrees
- moved IC1 43.8 mm to (36.8, 39.4), turned to 180 degrees
- moved G1 43.2 mm to (32.4, 24.1), flipped to the bottom, turned to 90 degrees
- moved C9 38.6 mm to (33.7, 45.1), turned to 270 degrees
- moved C6 35.8 mm to (42.5, 41.3), turned to 0 degrees
- moved L1 34.1 mm to (46.4, 41.4), turned to 180 degrees
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Connections:
- removed net PC10: IC1.51
- removed net PC11: IC1.52
- removed net PC12: IC1.53
- removed net U3_DE: IC4.2, IC4.3, R7.2
- removed net U3_RX: IC4.1
- removed net U3_TX: IC4.4
- new net DE3: IC1.53, IC4.4
- new net RXD3: IC1.52, IC4.1
- new net TXD3: IC1.51, IC4.2, IC4.3, R7.2
- net +3V3: now also R9.2
- net GND: now also JP2.1; no longer C15.2
- net RXD1: now also JP2.3, R9.1
- net TXD1: now also JP2.2
- net VBAT: no longer C15.1
Routing:
- net !RESET: track 51.3 -> 5.93 mm, vias 2 -> 0
- net BOOT0: track 37.1 -> 0.00 mm, vias 2 -> 0
- net DE3: track 0.00 -> 21.2 mm
- net TXD3: track 0.00 -> 14.8 mm
- net CAN_RX: track 0.00 -> 14.0 mm
- net +3V3: track 101.7 -> 115.2 mm
- net VBAT: track 0.00 -> 12.3 mm
- net RXD3: track 0.00 -> 12.3 mm
- net CAN_TX: track 0.00 -> 7.77 mm
- net BOOT1: track 17.4 -> 10.9 mm
- net OSC32_IN: track 15.5 -> 11.7 mm
- net N$44: track 8.72 -> 10.2 mm
- net OSC32_OUT: track 14.8 -> 13.7 mm
- net GND: vias 18 -> 19

Commit message: route timers
Parts:
- removed R17: 330, rc-master-smd:R0603
- added C15: 0.1, rc-master-smd:C0805
- added C18, C19: 100uF/6V3, rc-master-smd:SMC_D
- added R10, R11, R12, R22, R23, R24, R25, R26, R27, R28, R29, R30: 10, rc-master-smd:R0603
- added U1: (no value), vreg-linear:SOT223
- C14: device rc-master-smd:C0603 -> rc-master-smd:C0805
- Q1: device discrete:TC26H -> discrete:TC38H
- moved R19 57.8 mm to (14.0, 8.26)
- moved R18 57.8 mm to (14.0, 10.8)
- moved S1 57.8 mm to (6.35, 12.1)
- moved R16 42.5 mm to (9.53, 36.2), turned to 270 degrees
- moved C12 38.8 mm to (55.9, 36.2)
- moved R13 37.3 mm to (48.3, 36.2)
- moved R14 37.3 mm to (46.7, 36.2)
- moved R2 35.7 mm to (52.1, 29.8), turned to 90 degrees
- moved IC2 34.4 mm to (52.1, 36.2), turned to 180 degrees
- moved C4 31.3 mm to (29.2, 8.57), turned to 180 degrees
- moved JP1 30.6 mm to (83.8, 40.6)
- moved R4 30.6 mm to (79.4, 39.8)
- moved R6 30.6 mm to (78.7, 49.5)
- moved SW1 30.6 mm to (81.9, 36.8)
- moved C5 30.6 mm to (78.7, 47.5)
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Connections:
- removed net N$11: R17.2
- removed net N$14: R8.1
- new net N$15: R10.1, STMP1.2
- new net N$16: R11.1, STMP1.3
- new net N$17: R12.1, STMP1.4
- new net N$18: R22.1, STMP1.5
- new net N$19: R23.1, STMP1.7
- new net N$20: R24.1, STMP1.8
- new net N$21: R25.1, STMP1.9
- new net N$22: R26.1, STMP1.10
- new net N$23: R27.1, STMP1.12
- new net N$24: R28.1, STMP1.13
- new net N$25: R29.1, STMP1.14
- new net N$26: R30.1, STMP1.15
- net +3V3: now also C15.1, C19.+, U1.2; no longer C14.1
- net +5V: now also C14.1, C18.+, STMP1.20, U1.3
- net GND: now also C15.2, C18.-, C19.-, STMP1.1, STMP1.11, STMP1.19, STMP1.6, U1.1; no longer S1.2
- net N$8: now also R8.2; no longer R17.1
- net PC0: now also R27.2
- net PC1: now also R28.2
- net PC2: now also R29.2
- net PC3: now also R30.2
- net RS485_A: now also R8.1; no longer R8.2
- net RS485_B: now also S1.2
- net TIM3_CH1: now also R10.2
- net TIM3_CH2: now also R11.2
- net TIM3_CH3: now also R12.2
- net TIM3_CH4: now also R22.2
- net TIM4_CH1: now also R23.2
- net TIM4_CH2: now also R24.2
- net TIM4_CH3: now also R25.2
- net TIM4_CH4: now also R26.2
Routing:
- net TIM3_CH1: track 0.00 -> 66.1 mm, vias 0 -> 2
- net TIM3_CH2: track 0.00 -> 61.9 mm, vias 0 -> 2
- net TIM3_CH3: track 0.00 -> 56.0 mm, vias 0 -> 2
- net TIM3_CH4: track 0.00 -> 51.0 mm, vias 0 -> 2
- net CAN_L: track 5.77 -> 39.5 mm
- net TIM4_CH4: track 0.00 -> 31.3 mm
- net TIM4_CH3: track 0.00 -> 29.8 mm
- net TIM4_CH1: track 0.00 -> 28.9 mm
- net TIM4_CH2: track 0.00 -> 28.1 mm
- net RS485_B: track 5.77 -> 28.3 mm
- net PC0: track 0.00 -> 20.2 mm
- net PC3: track 0.00 -> 18.1 mm
- net PC1: track 0.00 -> 17.6 mm
- net N$2: track 4.50 -> 21.4 mm, vias 0 -> 2
- net PC2: track 0.00 -> 16.1 mm
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Other:
- board size 63.5 x 57.1 mm -> 69.8 x 57.1 mm

Commit message: route in progress
Parts:
- removed JP1: (no value), pinhead-fixdrills:1X02
- added R34, R37: 560, rc-master-smd:R0603
- added SW2: KSS-2EG4430, buttons:KSS-2EG4430
- Q1: device discrete:TC38H -> crystal:TC38H-G
- moved C16 45.6 mm to (78.7, 37.8), turned to 0 degrees
- moved R1 24.9 mm to (59.1, 47.6), turned to 0 degrees
- moved SW1 23.3 mm to (62.9, 50.2), turned to 270 degrees
- moved R3 20.7 mm to (58.7, 40.6), turned to 90 degrees
- moved LED1 19.3 mm to (59.7, 50.2), turned to 0 degrees
- moved R4 19.1 mm to (60.3, 40.6), turned to 90 degrees
- moved C5 18.7 mm to (60.3, 44.1)
- moved R6 16.2 mm to (63.5, 44.1), turned to 0 degrees
- moved R9 15.9 mm to (64.8, 18.4), turned to 270 degrees
- moved C17 9.23 mm to (63.5, 41.6)
- moved R21 8.60 mm to (63.5, 39.7)
- moved R8 8.26 mm to (13.3, 14.6)
- moved R20 7.65 mm to (63.5, 38.1)
- moved JP2 7.62 mm to (67.3, 22.2)
- moved JP4 7.62 mm to (67.3, 38.1)
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Connections:
- removed net N$12: R18.2
- removed net N$13: R19.2
- removed net N$25: R29.1, STMP1.14
- removed net N$26: R30.1, STMP1.15
- removed net PB5: IC1.57
- new net N$11: R27.1, STMP1.11
- new net N$14: R28.1, STMP1.12
- new net SW3: IC1.55, R18.2
- new net SW4: IC1.56, R19.2
- net +3V3: now also JP2.5, SW2.2; no longer JP1.1
- net +5V: now also JP2.4, R34.2
- net BOOT0: now also IC1.57
- net GND: now also Q1.GND, R37.1, STMP1.10; no longer STMP1.11, STMP1.6
- net N$19: now also STMP1.6; no longer STMP1.7
- net N$20: now also STMP1.7; no longer STMP1.8
- net N$21: now also STMP1.8; no longer STMP1.9
- net N$22: now also STMP1.9; no longer STMP1.10
- net N$23: now also R29.1, STMP1.13; no longer R27.1, STMP1.12
- net N$24: now also R30.1, STMP1.14; no longer R28.1, STMP1.13
- net N$3: now also SW2.1; no longer JP1.2
- net N$44: now also R34.1
- net N$6: now also R37.2
Routing:
- net !RESET: track 5.93 -> 44.1 mm, vias 0 -> 1
- net BOOT0: track 0.00 -> 20.7 mm, vias 0 -> 1
- net N$3: track 4.00 -> 17.1 mm, vias 0 -> 2
- net DE3: track 19.6 -> 8.02 mm
- net CAN_TX: track 22.8 -> 14.6 mm
- net N$8: track 10.7 -> 2.79 mm
- net CAN_RX: track 22.9 -> 15.1 mm
- net OSC32_IN: track 12.9 -> 7.13 mm
- net +3V3: track 109.0 -> 103.3 mm
- net RXD3: track 11.9 -> 17.6 mm
- net TIM3_CH3: track 56.0 -> 50.6 mm
- net TIM3_CH1: track 66.1 -> 60.7 mm
- net TIM3_CH2: track 61.9 -> 56.7 mm
- net CAN_H: track 8.48 -> 12.4 mm
- net PC0: track 20.2 -> 16.4 mm
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Other:
- board text added: "RST"
- board text added: "SYS"

Commit message: some pcb changes
Routing:
- net RXD1: track 0.00 -> 40.6 mm, vias 0 -> 1
- net TXD1: track 0.00 -> 37.3 mm, vias 0 -> 1
- net SW4: track 0.00 -> 27.2 mm
- net SW3: track 0.00 -> 25.8 mm
- net SWCLK: track 3.17 -> 14.7 mm, vias 0 -> 1
- net SWDIO: track 3.32 -> 12.8 mm, vias 0 -> 1
- net N$9: track 0.00 -> 2.56 mm
- net N$10: track 0.00 -> 2.56 mm
Changed lines of the file:
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@@
 <contactref element="IC1" pad="42"/>
 <contactref element="JP2" pad="2"/>
-<wire x1="36.715" y1="32.37" x2="67.31" y2="24.765" width="0" layer="19" extent="1-1"/>
+<wire x1="36.715" y1="32.37" x2="36.715" y2="31.38875" width="0.2032" layer="1"/>
+<wire x1="36.715" y1="31.38875" x2="37.1475" y2="30.95625" width="0.2032" layer="1"/>
+<via x="37.1475" y="30.95625" extent="1-16" drill="0.4"/>
+<wire x1="37.1475" y1="30.95625" x2="39.21125" y2="30.95625" width="0.2032" layer="16"/>
+<wire x1="39.21125" y1="30.95625" x2="40.005" y2="31.75" width="0.2032" layer="16"/>
+<wire x1="40.005" y1="31.75" x2="64.29375" y2="31.75" width="0.2032" layer="16"/>
+<wire x1="64.29375" y1="31.75" x2="65.405" y2="30.63875" width="0.2032" layer="16"/>
+<wire x1="65.405" y1="30.63875" x2="65.405" y2="26.67" width="0.2032" layer="16"/>
+<wire x1="65.405" y1="26.67" x2="67.31" y2="24.765" width="0.2032" layer="16"/>
 </signal>
 <signal name="RXD1">
@@
 <contactref element="JP2" pad="3"/>
 <contactref element="R9" pad="1"/>
-<wire x1="64.77" y1="19.177" x2="67.31" y2="22.225" width="0" layer="19" extent="1-1"/>
-<wire x1="36.215" y1="32.37" x2="64.77" y2="19.177" width="0" layer="19" extent="1-1"/>
+<wire x1="36.215" y1="32.37" x2="36.215" y2="30.61875" width="0.2032" layer="1"/>
+<wire x1="36.215" y1="30.61875" x2="36.67125" y2="30.1625" width="0.2032" layer="1"/>
+<wire x1="36.67125" y1="30.1625" x2="37.7825" y2="30.1625" width="0.2032" layer="1"/>
+<via x="37.7825" y="30.1625" extent="1-16" drill="0.4"/>
+<wire x1="37.7825" y1="30.1625" x2="38.1" y2="30.48" width="0.2032" layer="16"/>
+<wire x1="38.1" y1="30.48" x2="39.37" y2="30.48" width="0.2032" layer="16"/>
+<wire x1="39.37" y1="30.48" x2="40.16375" y2="31.27375" width="0.2032" layer="16"/>
+<wire x1="40.16375" y1="31.27375" x2="63.97625" y2="31.27375" width="0.2032" layer="16"/>
+<wire x1="63.97625" y1="31.27375" x2="64.92875" y2="30.32125" width="0.2032" layer="16"/>
+<wire x1="64.92875" y1="30.32125" x2="64.92875" y2="26.51125" width="0.2032" layer="16"/>
+<wire x1="64.92875" y1="26.51125" x2="66.04" y2="25.4" width="0.2032" layer="16"/>
+<wire x1="66.04" y1="25.4" x2="66.04" y2="23.495" width="0.2032" layer="16"/>
+<wire x1="66.04" y1="23.495" x2="67.31" y2="22.225" width="0.2032" layer="16"/>
+<wire x1="67.31" y1="22.225" x2="64.77" y2="19.177" width="0" layer="19" extent="1-1"/>
 </signal>
 <signal name="PB0">
@@
 <contactref element="R18" pad="1"/>
 <contactref element="S1" pad="6"/>
-<wire x1="10.65" y1="10.795" x2="13.208" y2="10.795" width="0" layer="19" extent="1-1"/>
+<wire x1="13.208" y1="10.795" x2="10.65" y2="10.795" width="0.2032" layer="1"/>
 </signal>
 <signal name="N$10">
 <contactref element="R19" pad="1"/>
 <contactref element="S1" pad="5"/>
-<wire x1="10.65" y1="8.255" x2="13.208" y2="8.255" width="0" layer="19" extent="1-1"/>
+<wire x1="10.65" y1="8.255" x2="13.208" y2="8.255" width="0.2032" layer="1"/>
 </signal>
 <signal name="SWDIO">
@@
 <wire x1="64.262" y1="39.6875" x2="66.2305" y2="39.6875" width="0.254" layer="1"/>
 <wire x1="66.2305" y1="39.6875" x2="67.183" y2="40.64" width="0.254" layer="1"/>
-<wire x1="34.715" y1="32.37" x2="64.262" y2="39.6875" width="0" layer="19" extent="1-1"/>
+<wire x1="34.715" y1="32.37" x2="34.715" y2="33.865" width="0.2032" layer="1"/>
+<wire x1="34.715" y1="33.865" x2="34.29" y2="34.29" width="0.2032" layer="1"/>
+<wire x1="34.29" y1="34.29" x2="34.13125" y2="34.29" width="0.2032" layer="1"/>
+<via x="34.13125" y="34.29" extent="1-16" drill="0.4"/>
+<wire x1="34.13125" y1="34.29" x2="34.6075" y2="34.29" width="0.2032" layer="16"/>
+<wire x1="34.6075" y1="34.29" x2="35.2425" y2="34.925" width="0.2032" layer="16"/>
+<wire x1="35.2425" y1="34.925" x2="35.2425" y2="40.3225" width="0.2032" layer="16"/>
+<wire x1="35.2425" y1="40.3225" x2="35.56" y2="40.64" width="0.2032" layer="16"/>
+<wire x1="35.56" y1="40.64" x2="64.262" y2="39.6875" width="0" layer="19" extent="1-16"/>
 </signal>
 <signal name="SWCLK">
@@
 <contactref element="R20" pad="1"/>
 <wire x1="67.437" y1="38.1" x2="64.262" y2="38.1" width="0.254" layer="1"/>
-<wire x1="31.765" y1="30.42" x2="64.262" y2="38.1" width="0" layer="19" extent="1-1"/>
+<wire x1="31.765" y1="30.42" x2="31.765" y2="31.1" width="0.2032" layer="1"/>
+<wire x1="31.765" y1="31.1" x2="31.75" y2="31.115" width="0.2032" layer="1"/>
+<wire x1="31.75" y1="31.115" x2="31.75" y2="32.385" width="0.2032" layer="1"/>
+<via x="33.02" y="34.29" extent="1-16" drill="0.4"/>
+<wire x1="33.02" y1="34.29" x2="33.655" y2="34.925" width="0.2032" layer="16"/>
+<wire x1="33.655" y1="34.925" x2="33.81375" y2="34.925" width="0.2032" layer="16"/>
+<wire x1="33.81375" y1="34.925" x2="34.76625" y2="35.8775" width="0.2032" layer="16"/>
+<wire x1="34.76625" y1="35.8775" x2="34.76625" y2="40.48125" width="0.2032" layer="16"/>
+<wire x1="34.76625" y1="40.48125" x2="34.925" y2="40.64" width="0.2032" layer="16"/>
+<wire x1="33.02" y1="34.29" x2="32.385" y2="33.655" width="0.2032" layer="1"/>
+<wire x1="32.385" y1="33.655" x2="31.75" y2="32.385" width="0.2032" layer="1" curve="36.869898"/>
+<wire x1="34.925" y1="40.64" x2="64.262" y2="38.1" width="0" layer="19" extent="1-16"/>
 </signal>
 <signal name="DE3">
@@
 <contactref element="IC1" pad="55"/>
 <contactref element="R18" pad="2"/>
-<wire x1="14.732" y1="10.795" x2="31.765" y2="27.42" width="0" layer="19" extent="1-1"/>
+<wire x1="26.908125" y1="25.796875" x2="23.098125" y2="21.986875" width="0.2032" layer="1"/>
+<wire x1="17.30375" y1="16.35125" x2="17.30375" y2="12.85875" width="0.2032" layer="1"/>
+<wire x1="17.30375" y1="16.35125" x2="20.32" y2="20.32" width="0.2032" layer="1" curve="-74.469681"/>
+<wire x1="20.32" y1="20.32" x2="23.098125" y2="21.986875" width="0.2032" layer="1" curve="30.86683"/>
+<wire x1="31.765" y1="27.42" x2="30.75375" y2="27.42" width="0.2032" layer="1"/>
+<wire x1="30.75375" y1="27.42" x2="26.908125" y2="25.796875" width="0.2032" layer="1" curve="45.766355"/>
+<wire x1="17.30375" y1="12.85875" x2="16.51" y2="11.43" width="0.2032" layer="1" curve="-58.109208"/>
+<wire x1="16.51" y1="11.43" x2="14.732" y2="10.795" width="0.2032" layer="1" curve="-24.47394"/>
 </signal>
 <signal name="SW4">
 <contactref element="IC1" pad="56"/>
 <contactref element="R19" pad="2"/>
-<wire x1="14.732" y1="8.255" x2="31.765" y2="26.92" width="0" layer="19" extent="1-1"/>
+<wire x1="27.225625" y1="25.479375" x2="23.733125" y2="21.986875" width="0.2032" layer="1"/>
+<wire x1="17.78" y1="16.35125" x2="17.78" y2="12.85875" width="0.2032" layer="1"/>
+<wire x1="17.78" y1="16.35125" x2="20.32" y2="19.84375" width="0.2032" layer="1" curve="-72.054747"/>
+<wire x1="20.32" y1="19.84375" x2="23.733125" y2="21.986875" width="0.2032" layer="1" curve="28.359541"/>
+<wire x1="31.765" y1="26.92" x2="30.73" y2="26.92" width="0.2032" layer="1"/>
+<wire x1="30.73" y1="26.92" x2="27.225625" y2="25.479375" width="0.2032" layer="1" curve="44.694469"/>
+<wire x1="17.78" y1="12.85875" x2="16.35125" y2="10.795" width="0.2032" layer="1" curve="-69.390273"/>
+<wire x1="16.35125" y1="10.795" x2="15.24" y2="9.525" width="0.2032" layer="1" curve="56.408866"/>
+<wire x1="15.24" y1="9.525" x2="14.732" y2="8.255" width="0.2032" layer="1" curve="-17.639834"/>
 </signal>
 </signals>
