File: pcb/stm32-40.brd (EAGLE design)
At the start: 69.8 x 57.1 mm, 82 parts, among them IC1 STM32F103RBT6, IC2 CAT24M01WI-GT3, IC3 AMIS30663CANG2G, IC4 MAX487-S, Q1 32768Hz, Q2 8MHz, SW1 KSS-2EG4430, SW2 KSS-2EG4430, X1 MCV3, X2 MCV3

Commit message: pcb in progress
Parts:
- removed C13: 0.1, rc-master-smd:C0603
- removed C24, C25: 560pF, rc-master-smd:C0603
- removed R37: 560, rc-master-smd:R0603
- removed R38: NC, rc-master-smd:R0603
- added C20: 0.1, rc-master-smd:C0603
- added C23: 560pF, rc-master-smd:C0603
- added LED2: (no value), led:CHIP-LED0805
- added R17: 10, rc-master-smd:R0603
- added R31: 330, rc-master-smd:R0603
- added R33: 100, rc-master-smd:R0603
- C14: value 0.1 -> 100uF/6V3; device rc-master-smd:C0805 -> rc-master-smd:SMC_D
- C16: value 0.1 -> 100uF/6V3; device rc-master-smd:C0603 -> rc-master-smd:SMC_D
- C17: device rc-master-smd:C0603 -> rc-master-smd:C0805
- C18, C19: value 100uF/6V3 -> 0.1; device rc-master-smd:SMC_D -> rc-master-smd:C0603
- C22: value 0.1 -> 560pF
- IC3: value AMIS30663CANG2G -> MAX487-S; device interfaces:SO08 -> rs232-rs485:SO08
- IC4: value MAX487-S -> AMIS30663CANG2G; device rs232-rs485:SO08 -> interfaces:SO08
- R10, R26: value 10 -> 10K
- R11, R12: value 10 -> 4.7K
- R13, R14: value 4.7K -> 10
- R15: value 100 -> 10
- R16: value 120 -> 10; device rc-master-smd:R0805 -> rc-master-smd:R0603
- R18, R19: value 330 -> 10
- R2: value 10K -> 220
- R20, R21: value 10K -> 10
- R25, R27: value 10 -> 560
- R28, R30: value 10 -> 120; device rc-master-smd:R0603 -> rc-master-smd:R0805
- R29: value 10 -> 330
- R34: value 560 -> 100
- R36: value 100 -> NC
- R4: value 2.2K -> 10K
- R5: value 1M -> 10K
- R6: value 10K -> 2.2K
- R7: value 10K -> 1M
- R8: value 120 -> 10K; device rc-master-smd:R0805 -> rc-master-smd:R0603
- moved R10 62.5 mm to (63.5, 39.7)
- moved R8 58.2 mm to (63.5, 44.1), turned to 0 degrees
- moved R11 51.8 mm to (59.1, 31.8), turned to 0 degrees
- moved R12 50.0 mm to (59.1, 33.3)
- moved C7 48.2 mm to (63.5, 41.6), turned to 180 degrees
- moved R13 45.4 mm to (11.4, 5.08), turned to 180 degrees
- moved R30 44.8 mm to (10.8, 32.4)
- moved R20 44.5 mm to (33.7, 5.08)
- moved R21 43.7 mm to (36.8, 5.08)
- moved R14 42.0 mm to (14.6, 5.08), turned to 180 degrees
- moved C18 40.4 mm to (18.7, 23.8), turned to 0 degrees
- moved LED1 39.4 mm to (66.7, 11.4), turned to 270 degrees
- moved C19 37.5 mm to (21.6, 33.7), turned to 270 degrees
- moved C16 37.1 mm to (51.4, 12.7), turned to 270 degrees
- moved C17 36.1 mm to (59.7, 5.71)
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- renumbered JP4 to JP1
Connections:
- new net N$30: LED2.A, R2.2
- net !RESET: now also R8.1, SW2.2; no longer R6.1, SW1.2
- net +3V3: now also C16.+, C20.1, C7.1, R1.1, R10.2, R11.2, R12.2, R5.2, R8.2, SW1.2; no longer C17.1, C19.+, C22.1, R13.2, R14.2, R20.2, R21.2, R6.2, SW2.2
- net +5V: now also C14.+, C17.1, C18.1, C19.1, IC3.8, IC4.3, R25.2; no longer C14.1, C18.+, C21.1, C7.1, IC3.3, IC4.8, R34.2
- net BOOT0: now also R4.1; no longer R3.1
- net BOOT1: now also R3.1; no longer R1.1
- net CAN_CTRL: now also IC4.8, R36.2; no longer IC3.8, R38.2
- net CAN_H: now also F3.P$2, R30.1, X2.1; no longer F2.P$2, R16.1, X1.1
- net CAN_L: now also F4.P$2, X2.3; no longer F3.P$2, X1.3
- net CAN_RX: now also R33.1; no longer R15.1
- net CAN_TX: now also IC4.1; no longer IC3.1
- net DE3: now also IC3.4; no longer IC4.4
- net GND: now also C14.-, C16.-, C18.2, C19.2, C20.2, C23.2, IC3.5, IC4.2, LED2.C, R26.1, R27.1, R3.2, R36.1, R6.1, STMP1.21, STMP1.40, SW2.1; no longer C13.2, C14.2, C16.2, C18.-, C19.-, C24.2, C25.2, IC3.2, IC4.5, R2.2, R37.1, R38.1, R4.1, R7.1, SW1.1
- net N$1: now also C21.1, IC4.5; no longer C13.1, IC3.5
- net N$10: now also R31.1; no longer R19.1
- net N$11: now also R21.1; no longer R27.1
- net N$14: now also R22.1; no longer R28.1
- net N$15: now also R13.1; no longer R10.1
- net N$16: now also R14.1; no longer R11.1
- net N$17: now also R15.1; no longer R12.1
- net N$18: now also R16.1; no longer R22.1
- net N$19: now also R17.1; no longer R23.1
- net N$2: now also R30.2; no longer R16.2
- net N$20: now also R18.1; no longer R24.1
- net N$21: now also R19.1; no longer R25.1
- net N$22: now also R20.1; no longer R26.1
- net N$23: now also R23.1; no longer R29.1
- net N$24: now also R24.1; no longer R30.1
- net N$3: now also R6.2, SW1.1; no longer R3.2, SW2.1
- net N$44: now also F2.P$1, IC3.6, R25.1; no longer F4.P$1, IC4.6, R34.1
- net N$51: now also F3.P$1, IC4.7, R34.2; no longer F2.P$1, IC3.7, R35.2
- net N$52: now also F4.P$1, IC4.6, R35.2; no longer F3.P$1, IC3.6, R36.2
- net N$54: now also C23.1, R35.1; no longer C25.1, R36.1
- net N$55: now also C22.1, R34.1; no longer C24.1, R35.1
- net N$6: now also IC3.7, R27.2; no longer IC4.7, R37.2
- net N$7: now also IC4.4, R33.2; no longer IC3.4, R15.2
- net N$8: now also R28.2; no longer R8.2
- net N$9: now also R29.1; no longer R18.1
- net OSC_IN: now also R7.2; no longer R5.2
- net OSC_OUT: now also R7.1; no longer R5.1
- net PC0: now also R21.2; no longer R27.2
- net PC1: now also R22.2; no longer R28.2
- net PC13: now also STMP1.39
- net PC2: now also R23.2; no longer R29.2
- net PC3: now also R24.2; no longer R30.2
- net RS485_A: now also F2.P$2, R28.1, X1.1; no longer F4.P$2, R8.1, X2.1
- net RS485_B: now also X1.3; no longer X2.3
- net RXD1: now also R5.1; no longer R9.1
- net RXD3: now also IC3.1; no longer IC4.1
- net SCL2: now also R11.1; no longer R13.1
- net SDA2: now also R12.1; no longer R14.1
- net SW3: now also R29.2; no longer R18.2
- net SW4: now also R31.2; no longer R19.2
- net SWCLK: now also R9.1; no longer R20.1
- net SWDIO: now also R10.1; no longer R21.1
- net TIM3_CH1: now also R13.2; no longer R10.2
- net TIM3_CH2: now also R14.2; no longer R11.2
- net TIM3_CH3: now also R15.2; no longer R12.2
- net TIM3_CH4: now also R16.2; no longer R22.2
- net TIM4_CH1: now also R17.2; no longer R23.2
- net TIM4_CH2: now also R18.2; no longer R24.2
- net TIM4_CH3: now also R19.2; no longer R25.2
- net TIM4_CH4: now also R20.2; no longer R26.2
- net TXD3: now also IC3.2, IC3.3, R26.2; no longer IC4.2, IC4.3, R7.2
- net VDDA: no longer C16.1
Routing:
- net PC13: track 0.00 -> 55.1 mm, vias 0 -> 1
- net SWCLK: track 14.7 -> 50.5 mm
- net SWDIO: track 12.8 -> 44.1 mm, vias 1 -> 2
- net BOOT0: track 20.7 -> 49.3 mm, vias 1 -> 2
- net !RESET: track 44.1 -> 70.1 mm, vias 1 -> 2
- net N$30: track 0.00 -> 10.0 mm
- net SCL2: track 11.3 -> 4.20 mm
- net SDA2: track 11.2 -> 4.94 mm
- net RXD1: track 40.6 -> 44.3 mm
- net N$3: track 17.1 -> 20.4 mm
- net TIM3_CH1: track 60.7 -> 58.5 mm
- net TIM3_CH2: track 56.7 -> 54.5 mm
- net N$52: track 10.2 -> 12.2 mm
- net TIM4_CH3: track 32.5 -> 30.6 mm
- net TIM3_CH4: track 48.2 -> 46.4 mm
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Other:
- board text added: "Pwr"
- board text added: "Stat"

Commit message: pcb in progress
Connections:
- net PA0: now also STMP1.22
- net PA1: now also STMP1.23
- net PA2: now also STMP1.24
- net PA3: now also STMP1.25
- net PA4: now also STMP1.26
- net PA5: now also STMP1.27
- net PA6: now also STMP1.28
- net PA7: now also STMP1.29
Routing:
- net PA0: track 0.00 -> 47.8 mm
- net PA1: track 0.00 -> 45.0 mm
- net PA7: track 0.00 -> 44.7 mm
- net PA6: track 0.00 -> 43.6 mm
- net PA2: track 0.00 -> 42.7 mm
- net PA5: track 0.00 -> 42.4 mm
- net PA4: track 0.00 -> 41.3 mm
- net PA3: track 0.00 -> 40.8 mm
- net +3V3: track 102.3 -> 103.1 mm
Changed lines of the file:
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@@
 <contactref element="C16" pad="+"/>
 <wire x1="43.942" y1="23.495" x2="45.085" y2="23.495" width="0.6096" layer="16"/>
-<wire x1="43.942" y1="23.495" x2="43.942" y2="20.4469" width="0.6096" layer="16"/>
-<wire x1="43.942" y1="20.4469" x2="40.6401" y2="17.145" width="0.6096" layer="16"/>
+<wire x1="43.942" y1="23.495" x2="43.942" y2="22.352" width="0.6096" layer="16"/>
+<wire x1="43.942" y1="22.352" x2="43.18" y2="21.59" width="0.6096" layer="16"/>
+<wire x1="40.6401" y1="17.1451" x2="40.6401" y2="17.145" width="0.6096" layer="16"/>
 <wire x1="41.9101" y1="15.875" x2="40.6401" y2="17.145" width="0.6096" layer="1"/>
 <contactref element="SW1" pad="2"/>
@@
 <wire x1="33.655" y1="20.955" x2="37.7825" y2="18.415" width="0.6096" layer="16" curve="-63.215004"/>
 <wire x1="37.7825" y1="18.415" x2="40.6401" y2="17.145" width="0.6096" layer="16" curve="78.506456"/>
+<wire x1="43.18" y1="21.59" x2="41.91" y2="21.59" width="0.6096" layer="16"/>
+<wire x1="41.91" y1="21.59" x2="41.275" y2="20.955" width="0.6096" layer="16"/>
+<wire x1="41.275" y1="20.955" x2="41.275" y2="17.7799" width="0.6096" layer="16"/>
+<wire x1="41.275" y1="17.7799" x2="40.6401" y2="17.145" width="0.6096" layer="16"/>
 <wire x1="59.817" y1="33.3375" x2="62.738" y2="38.1" width="0" layer="19" extent="1-1"/>
 <wire x1="64.77" y1="27.432" x2="59.817" y2="28.86075" width="0" layer="19" extent="1-1"/>
 <wire x1="52.451" y1="18.415" x2="58.293" y2="24.13" width="0" layer="19" extent="1-1"/>
-<wire x1="43.942" y1="20.4469" x2="52.451" y2="18.415" width="0" layer="19" extent="1-16"/>
+<wire x1="45.085" y1="23.495" x2="52.451" y2="18.415" width="0" layer="19" extent="1-1"/>
 <wire x1="19.05" y1="32.893" x2="32.86125" y2="33.02" width="0" layer="19" extent="1-1"/>
 </signal>
@@
 <signal name="PA0">
 <contactref element="IC1" pad="14"/>
+<contactref element="STMP1" pad="22"/>
+<wire x1="40.215" y1="20.97" x2="40.215" y2="19.95125" width="0.2032" layer="1"/>
+<wire x1="40.215" y1="19.95125" x2="40.64" y2="19.52625" width="0.2032" layer="1"/>
+<wire x1="40.64" y1="19.52625" x2="41.75125" y2="19.52625" width="0.2032" layer="1"/>
+<wire x1="41.75125" y1="19.52625" x2="42.2275" y2="20.0025" width="0.2032" layer="1"/>
+<wire x1="42.2275" y1="20.0025" x2="44.7675" y2="20.0025" width="0.2032" layer="1"/>
+<wire x1="44.7675" y1="20.0025" x2="47.3075" y2="22.5425" width="0.2032" layer="1"/>
+<wire x1="47.3075" y1="22.5425" x2="50.64125" y2="22.5425" width="0.2032" layer="1"/>
+<wire x1="50.64125" y1="22.5425" x2="53.49875" y2="25.4" width="0.2032" layer="1"/>
+<wire x1="53.49875" y1="25.4" x2="53.49875" y2="52.3875" width="0.2032" layer="1"/>
+<wire x1="53.49875" y1="52.3875" x2="55.72125" y2="54.61" width="0.2032" layer="1"/>
+<wire x1="55.72125" y1="54.61" x2="56.515" y2="54.61" width="0.2032" layer="1"/>
 </signal>
 <signal name="PA8">
@@
 <signal name="PA4">
 <contactref element="IC1" pad="20"/>
+<contactref element="STMP1" pad="26"/>
+<wire x1="43.165" y1="24.42" x2="49.97875" y2="24.42" width="0.2032" layer="1"/>
+<wire x1="49.97875" y1="24.42" x2="51.59375" y2="26.035" width="0.2032" layer="1"/>
+<wire x1="51.59375" y1="26.035" x2="51.59375" y2="51.91125" width="0.2032" layer="1"/>
+<wire x1="51.59375" y1="51.91125" x2="50.165" y2="53.34" width="0.2032" layer="1"/>
+<wire x1="50.165" y1="53.34" x2="47.625" y2="53.34" width="0.2032" layer="1"/>
+<wire x1="47.625" y1="53.34" x2="46.355" y2="54.61" width="0.2032" layer="1"/>
 </signal>
 <signal name="PA5">
 <contactref element="IC1" pad="21"/>
+<contactref element="STMP1" pad="27"/>
+<wire x1="43.165" y1="24.92" x2="49.84375" y2="24.92" width="0.2032" layer="1"/>
+<wire x1="49.84375" y1="24.92" x2="51.1175" y2="26.19375" width="0.2032" layer="1"/>
+<wire x1="51.1175" y1="26.19375" x2="51.1175" y2="51.59375" width="0.2032" layer="1"/>
+<wire x1="51.1175" y1="51.59375" x2="49.8475" y2="52.86375" width="0.2032" layer="1"/>
+<wire x1="49.8475" y1="52.86375" x2="46.51375" y2="52.86375" width="0.2032" layer="1"/>
+<wire x1="46.51375" y1="52.86375" x2="44.7675" y2="54.61" width="0.2032" layer="1"/>
+<wire x1="44.7675" y1="54.61" x2="43.815" y2="54.61" width="0.2032" layer="1"/>
 </signal>
 <signal name="PA6">
 <contactref element="IC1" pad="22"/>
+<contactref element="STMP1" pad="28"/>
+<wire x1="43.165" y1="25.42" x2="49.70875" y2="25.42" width="0.2032" layer="1"/>
+<wire x1="49.70875" y1="25.42" x2="50.64125" y2="26.3525" width="0.2032" layer="1"/>
+<wire x1="50.64125" y1="26.3525" x2="50.64125" y2="51.435" width="0.2032" layer="1"/>
+<wire x1="50.64125" y1="51.435" x2="49.68875" y2="52.3875" width="0.2032" layer="1"/>
+<wire x1="49.68875" y1="52.3875" x2="46.0375" y2="52.3875" width="0.2032" layer="1"/>
+<wire x1="46.0375" y1="52.3875" x2="45.085" y2="53.34" width="0.2032" layer="1"/>
+<wire x1="45.085" y1="53.34" x2="43.33875" y2="53.34" width="0.2032" layer="1"/>
+<wire x1="43.33875" y1="53.34" x2="42.06875" y2="54.61" width="0.2032" layer="1"/>
+<wire x1="42.06875" y1="54.61" x2="41.275" y2="54.61" width="0.2032" layer="1"/>
 </signal>
 <signal name="PA7">
 <contactref element="IC1" pad="23"/>
+<contactref element="STMP1" pad="29"/>
+<wire x1="43.165" y1="25.92" x2="49.57375" y2="25.92" width="0.2032" layer="1"/>
+<wire x1="49.57375" y1="25.92" x2="50.165" y2="26.51125" width="0.2032" layer="1"/>
+<wire x1="50.165" y1="26.51125" x2="50.165" y2="51.1175" width="0.2032" layer="1"/>
+<wire x1="50.165" y1="51.1175" x2="49.37125" y2="51.91125" width="0.2032" layer="1"/>
+<wire x1="49.37125" y1="51.91125" x2="45.72" y2="51.91125" width="0.2032" layer="1"/>
+<wire x1="45.72" y1="51.91125" x2="44.7675" y2="52.86375" width="0.2032" layer="1"/>
+<wire x1="44.7675" y1="52.86375" x2="41.275" y2="52.86375" width="0.2032" layer="1"/>
+<wire x1="41.275" y1="52.86375" x2="39.52875" y2="54.61" width="0.2032" layer="1"/>
+<wire x1="39.52875" y1="54.61" x2="38.735" y2="54.61" width="0.2032" layer="1"/>
 </signal>
 <signal name="N$9">
@@
 <signal name="PA2">
 <contactref element="IC1" pad="16"/>
+<contactref element="STMP1" pad="24"/>
+<wire x1="41.215" y1="20.97" x2="44.465" y2="20.97" width="0.2032" layer="1"/>
+<wire x1="44.465" y1="20.97" x2="46.99" y2="23.495" width="0.2032" layer="1"/>
+<wire x1="46.99" y1="23.495" x2="50.32375" y2="23.495" width="0.2032" layer="1"/>
+<wire x1="50.32375" y1="23.495" x2="52.54625" y2="25.7175" width="0.2032" layer="1"/>
+<wire x1="52.54625" y1="25.7175" x2="52.54625" y2="53.49875" width="0.2032" layer="1"/>
+<wire x1="52.54625" y1="53.49875" x2="51.435" y2="54.61" width="0.2032" layer="1"/>
 </signal>
 <signal name="PA3">
 <contactref element="IC1" pad="17"/>
+<contactref element="STMP1" pad="25"/>
+<wire x1="43.165" y1="22.92" x2="44.54875" y2="22.92" width="0.2032" layer="1"/>
+<wire x1="44.54875" y1="22.92" x2="44.7675" y2="22.70125" width="0.2032" layer="1"/>
+<wire x1="44.7675" y1="22.70125" x2="45.56125" y2="22.70125" width="0.2032" layer="1"/>
+<wire x1="45.56125" y1="22.70125" x2="46.83125" y2="23.97125" width="0.2032" layer="1"/>
+<wire x1="46.83125" y1="23.97125" x2="50.165" y2="23.97125" width="0.2032" layer="1"/>
+<wire x1="50.165" y1="23.97125" x2="52.07" y2="25.87625" width="0.2032" layer="1"/>
+<wire x1="52.07" y1="25.87625" x2="52.07" y2="52.22875" width="0.2032" layer="1"/>
+<wire x1="52.07" y1="52.22875" x2="49.68875" y2="54.61" width="0.2032" layer="1"/>
+<wire x1="49.68875" y1="54.61" x2="48.895" y2="54.61" width="0.2032" layer="1"/>
 </signal>
 <signal name="PA1">
 <contactref element="IC1" pad="15"/>
+<contactref element="STMP1" pad="23"/>
+<wire x1="40.715" y1="20.97" x2="40.715" y2="20.08625" width="0.2032" layer="1"/>
+<wire x1="40.715" y1="20.08625" x2="40.79875" y2="20.0025" width="0.2032" layer="1"/>
+<wire x1="40.79875" y1="20.0025" x2="41.5925" y2="20.0025" width="0.2032" layer="1"/>
+<wire x1="41.5925" y1="20.0025" x2="42.06875" y2="20.47875" width="0.2032" layer="1"/>
+<wire x1="42.06875" y1="20.47875" x2="44.60875" y2="20.47875" width="0.2032" layer="1"/>
+<wire x1="44.60875" y1="20.47875" x2="47.14875" y2="23.01875" width="0.2032" layer="1"/>
+<wire x1="47.14875" y1="23.01875" x2="50.4825" y2="23.01875" width="0.2032" layer="1"/>
+<wire x1="50.4825" y1="23.01875" x2="53.0225" y2="25.55875" width="0.2032" layer="1"/>
+<wire x1="53.0225" y1="25.55875" x2="53.0225" y2="53.6575" width="0.2032" layer="1"/>
+<wire x1="53.0225" y1="53.6575" x2="53.975" y2="54.61" width="0.2032" layer="1"/>
 </signal>
 <signal name="RXD3">

Commit message: stamp + lcd
Parts:
- removed JP1: (no value), jtag:1X05
- added C13: 0.1, rc-master-smd:C0603
- added LCD1: (no value), lcd1202:NOKIA1202LCD-EXT
- added Q3: MMBT2222, semiconductor:SOT23
- added R37, R38, R39, R40, R43: 10, rc-master-smd:R0603
- added R41, R42: 4.7K, rc-master-smd:R0603
- added R44: 2K, rc-master-smd:R0603
- added SW3, SW4, SW5: KSS-2EG4430, buttons:KSS-2EG4430
- added SWD1: SWD-6, jtag:JTAG6PIN
- G1: device battery:LITHOLDER -> battery:SMT1220
- moved JP2 64.8 mm to (2.54, 21.6)
- moved SW1 64.8 mm to (2.54, 50.2)
- moved LED1 63.5 mm to (3.17, 10.8), turned to 90 degrees
- moved R1 63.5 mm to (3.17, 14.0), flipped to the bottom
- moved LED2 63.5 mm to (3.17, 7.62), turned to 90 degrees
- moved X1 61.0 mm to (65.4, 26.7), turned to 270 degrees
- moved X2 61.0 mm to (65.4, 42.5), turned to 270 degrees
- moved R2 59.7 mm to (5.08, 17.1), flipped to the bottom
- moved R5 59.7 mm to (5.08, 26.0), flipped to the bottom
- moved R10 57.2 mm to (6.35, 38.1), flipped to the bottom
- moved R9 57.2 mm to (6.35, 39.7), flipped to the bottom
- moved C7 57.1 mm to (6.35, 41.6), flipped to the bottom
- moved R8 57.1 mm to (6.35, 44.1), flipped to the bottom
- moved S1 57.1 mm to (63.5, 12.1)
- moved SW2 55.9 mm to (6.99, 50.2)
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- renumbered STMP1 to STMP2
Connections:
- new net !LCD_CS: LCD1.2, R41.1
- new net BL: R44.2
- new net LCD_CLK: LCD1.5
- new net LCD_DATA: LCD1.4
- new net N$25: R37.1, STMP2.6
- new net N$26: R38.1, STMP2.5
- new net N$27: R39.1, STMP2.4
- new net N$28: R40.1, STMP2.3
- new net N$29: LCD1.9, Q3.3
- new net N$31: LCD1.10, R43.1
- new net N$32: Q3.1, R44.1
- new net PA15: IC1.50, STMP2.24
- net !RESET: now also LCD1.1, R42.2, SWD1.5; no longer JP1.4
- net +3V3: now also C13.1, LCD1.6, LCD1.7, R41.2, R43.2, SWD1.1; no longer JP1.1
- net +5V: now also STMP2.1; no longer STMP2.20
- net CAN_L: now also S1.8, X2.2; no longer S1.1, X2.3
- net GND: now also C13.2, LCD1.3, LCD1.8, Q3.2, R42.1, S1.5, S1.6, STMP2.11, STMP2.2, STMP2.20, SW3.1, SW4.1, SW5.1, SWD1.3, X1.3, X2.3; no longer JP1.5, S1.3, S1.4, STMP2.1, STMP2.10, STMP2.19, X1.2, X2.2
- net N$10: now also S1.4; no longer S1.5
- net N$11: now also STMP2.10; no longer STMP2.11
- net N$14: now also STMP2.9; no longer STMP2.12
- net N$15: now also STMP2.19; no longer STMP2.2
- net N$16: now also STMP2.18; no longer STMP2.3
- net N$17: now also STMP2.17; no longer STMP2.4
- net N$18: now also STMP2.16; no longer STMP2.5
- net N$19: now also STMP2.15; no longer STMP2.6
- net N$2: now also S1.1; no longer S1.8
- net N$20: now also STMP2.14; no longer STMP2.7
- net N$21: now also STMP2.13; no longer STMP2.8
- net N$22: now also STMP2.12; no longer STMP2.9
- net N$23: now also STMP2.8; no longer STMP2.13
- net N$24: now also STMP2.7; no longer STMP2.14
- net N$8: now also S1.2; no longer S1.7
- net N$9: now also S1.3; no longer S1.6
- net PA0: now also STMP2.39; no longer STMP2.22
- net PA1: now also STMP2.38; no longer STMP2.23
- net PA2: now also STMP2.37; no longer STMP2.24
- net PA3: now also STMP2.36; no longer STMP2.25
- net PA4: now also STMP2.35; no longer STMP2.26
- net PA5: now also STMP2.34; no longer STMP2.27
- net PA6: now also STMP2.33; no longer STMP2.28
- net PA7: now also STMP2.32; no longer STMP2.29
- net PA8: now also STMP2.25
- net PB0: now also R39.2
- net PB1: now also R40.2
- net PC13: now also STMP2.22; no longer STMP2.39
- net PC4: now also R37.2
- net PC5: now also R38.2
- net PD2: now also STMP2.23
- net RS485_A: now also X1.2; no longer X1.1
- net RS485_B: now also S1.7, X1.1; no longer S1.2, X1.3
- net SCL2: now also STMP2.31
- net SDA2: now also STMP2.30
- net SPI2_MISO: now also STMP2.27
- net SPI2_MOSI: now also STMP2.26
- net SPI2_NSS: now also STMP2.29
- net SPI2_SCLK: now also STMP2.28
- net SWCLK: now also SWD1.2; no longer JP1.3
- net SWDIO: now also SWD1.4; no longer JP1.2
Routing:
- net SDA2: track 4.94 -> 60.2 mm, vias 0 -> 2
- net SCL2: track 4.20 -> 56.8 mm, vias 0 -> 2
- net PC13: track 55.1 -> 9.00 mm
- net PD2: track 0.00 -> 41.7 mm, vias 0 -> 2
- net PA15: track 0.00 -> 36.3 mm, vias 0 -> 2
- net PA8: track 0.00 -> 33.2 mm, vias 0 -> 2
- net SPI2_MOSI: track 0.00 -> 30.4 mm
- net SPI2_MISO: track 0.00 -> 28.5 mm
- net SPI2_SCLK: track 0.00 -> 27.3 mm
- net SPI2_NSS: track 0.00 -> 26.4 mm
- net PB0: track 0.00 -> 24.0 mm, vias 0 -> 2
- net PB1: track 0.00 -> 23.7 mm, vias 0 -> 2
- net PC5: track 0.00 -> 23.1 mm, vias 0 -> 2
- net PC4: track 0.00 -> 22.7 mm, vias 0 -> 2
- net N$25: track 0.00 -> 12.5 mm
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Other:
- board text added: "UART"
