File: pcb/stm32-d40-platform.sch (EAGLE design)
At the start: 84 parts, among them IC1 STM32F103C8, IC2 TODO AMIS30663CANG2G, IC3 STM32F103C8, J1 DIP-40, Q1 8MHz, Q2 8MHz, SW1 KSS-2EG4430, SW2 KSS-2EG4430, X1 DG3XX-03-3.5

Commit message: motherboard in progress
Parts:
- added 3V3, AVCC, PA0, PA1, PA10, PA11, PA12, PA13, PA14, PA15, PA2, PA3, PA4, PA5, PA6, PA7, PA8, PA9, PB0, PB1, PB10, PB11, PB12, PB13, PB14, PB15, PB2, PB3, PB4, PB5, PB6, PB7, PB8, PB9, PC14, PC15, RST, VBAT: (no value), pinhead-fixdrills:PIN-1X1_2.54
- added C23, C24: 22pF, rc-master-smd:C_0603
- added G1: B2430, battery:B2430
- added IC4: (no value), transistor-arrays:ULN2003D
- added K1, K2, K3, K4: ZNS5124, myrelays:ZNS5124
- added MOD1: STM32-MOD-CAN, stamp:STM32-MOD-CAN
- added Q3: 32768Hz, crystal:CRSTL3-
- added R36: 1M, rc-master-smd:R_0603
- added SG1: F/QMBIII, buzzer:F/QMBIII
- added X2: DG3XX-12-5.0, degson:DG3XX-12-5.0
- added X3: DG3XX-02-5.0, degson:DG3XX-02-5.0
Connections:
- new net !S2.RESET: MOD1.!RESET, RST.1
- new net N$366: IC4.15, K41.2
- new net N$367: IC4.14, K31.2
- new net N$368: IC4.13, K21.2
- new net N$369: IC4.12, K11.2
- new net N$370: IC4.16, SG1.+
- new net N$64: K12.S, X2-1.KL
- new net N$65: K12.P, X2-2.KL
- new net N$66: K12.O, X2-3.KL
- new net N$67: K22.S, X2-4.KL
- new net N$68: K22.P, X2-5.KL
- new net N$69: K22.O, X2-6.KL
- new net N$70: K32.S, X2-7.KL
- new net N$71: K32.P, X2-8.KL
- new net N$72: K32.O, X2-9.KL
- new net N$73: K42.S, X2-10.KL
- new net N$74: K42.P, X2-11.KL
- new net N$75: K42.O, X2-12.KL
- new net S2.3V3: 3V3.1, MOD1.+3V3
- new net S2.AVCC: AVCC.1, MOD1.AVCC
- new net S2.OSC32_IN: C24.1, MOD1.PC14, PC14.1, Q3.2, R36.2
- new net S2.OSC32_OUT: C23.1, MOD1.PC15, PC15.1, Q3.1, R36.1
- new net S2.PA0: MOD1.PA0, PA0.1
- new net S2.PA1: MOD1.PA1, PA1.1
- new net S2.PA10: MOD1.PA10, PA10.1
- new net S2.PA11: MOD1.PA11, PA11.1
- new net S2.PA12: MOD1.PA12, PA12.1
- new net S2.PA13: MOD1.PA13, PA13.1
- new net S2.PA14: MOD1.PA14, PA14.1
- new net S2.PA15: MOD1.PA15, PA15.1
- new net S2.PA2: MOD1.PA2, PA2.1
- new net S2.PA3: MOD1.PA3, PA3.1
- new net S2.PA4: MOD1.PA4, PA4.1
- new net S2.PA5: MOD1.PA5, PA5.1
- new net S2.PA6: MOD1.PA6, PA6.1
- new net S2.PA7: MOD1.PA7, PA7.1
- new net S2.PA8: MOD1.PA8, PA8.1
- new net S2.PA9: MOD1.PA9, PA9.1
- new net S2.PB0: MOD1.PB0, PB0.1
- new net S2.PB1: MOD1.PB1, PB1.1
- new net S2.PB10: MOD1.PB10, PB10.1
- new net S2.PB11: MOD1.PB11, PB11.1
- new net S2.PB12: MOD1.PB12, PB12.1
- new net S2.PB13: MOD1.PB13, PB13.1
- new net S2.PB14: MOD1.PB14, PB14.1
- new net S2.PB15: MOD1.PB15, PB15.1
- new net S2.PB2: MOD1.PB2, PB2.1
- new net S2.PB3: MOD1.PB3, PB3.1
- new net S2.PB4: MOD1.PB4, PB4.1
- new net S2.PB5: MOD1.PB5, PB5.1
- new net S2.PB6: MOD1.PB6, PB6.1
- new net S2.PB7: MOD1.PB7, PB7.1
- new net S2.PB8: MOD1.PB8, PB8.1
- new net S2.PB9: MOD1.PB9, PB9.1
- new net S2.VBAT: G1.+, MOD1.VBAT, VBAT.1
- net +5V: now also IC4.9, K11.1, K21.1, K31.1, K41.1, SG1.-, X3-2.KL
- net GND: now also C23.2, C24.2, G1.-, IC4.8, MOD1.GND@11, MOD1.GND@31, Q3.P$1, X3-1.KL

Commit message: PCB ready
Parts:
- removed SG1: F/QMBIII, buzzer:F/QMBIII
- added C25, C26: 0.1, rc-master-smd:C_0805
- added C27, C28: 100uF/6V3, rc-master:CP_E-035X080
- added D3: (no value), diodes:D-SMB
- added IN1, IN2, IN3, IN4, IN5, IN6, IN7, OUT5, OUT6, OUT7: (no value), pinhead-fixdrills:PIN-1X1_2.54
- added U2: (no value), vreg-linear:LM1117-3.3
- C23, C24: device rc-master-smd:C_0603 -> rc-master-smd:C_0805
- R36: device rc-master-smd:R_0603 -> rc-master-smd:R_0805
Connections:
- removed net N$370: IC4.16, SG1.+
- new net HEAT: U2.MASS
- new net N$11: D3.A, X3-2.KL
- new net S2.IN1: IC4.1, IN1.1
- new net S2.IN2: IC4.2, IN2.1
- new net S2.IN3: IC4.3, IN3.1
- new net S2.IN4: IC4.4, IN4.1
- new net S2.IN5: IC4.5, IN5.1
- new net S2.IN6: IC4.6, IN6.1
- new net S2.IN7: IC4.7, IN7.1
- new net S2.OUT5: IC4.12, OUT5.1
- new net S2.OUT6: IC4.11, OUT6.1
- new net S2.OUT7: IC4.10, OUT7.1
- net +5V: now also C25.1, C27.+, D3.C, U2.IN; no longer SG1.-, X3-2.KL
- net GND: now also C25.2, C26.2, C27.-, C28.-, U2.GND
- net N$366: now also IC4.13; no longer IC4.15
- net N$368: now also IC4.15; no longer IC4.13
- net N$369: now also IC4.16; no longer IC4.12
- net S2.3V3: now also C26.1, C28.+, U2.OUT
Other:
- moved on the sheet: IC4

Commit message: ST-link v2 SWD some fixes
Parts:
- removed D2: (no value), diodes:BAT54A1-C3
- removed R31: 10K, rc-master-smd:R_0603
- removed R32: 100, rc-master-smd:R_0603
- added C29: 0.01, rc-master-smd:C_0603
- added R37: 220, rc-master-smd:R_0603
- added R38: 4.7K, rc-master-smd:R_0603
- R19: value 100 -> 220
- R26, R27: value 0 -> 22
- R34, R35: value 100 -> 510
Connections:
- removed net N$49: D2.C, R32.2
- new net S3.M25_CS: IC3.PA1/USART2_RTS/ADC12_IN1/TIM2_CH2
- new net S3.U2_CK: IC3.PA4/SPI1_NSS/ADC12_IN4/USART2_CK
- new net S3.U2_RX: IC3.PA3/USART2_RX/ADC12_IN3/TIM2_CH4
- new net S3.U2_TX: IC3.PA2/USART2_TX/ADC12_IN2/TIM2_CH3
- net +3V3: now also R38.2; no longer D2.A, R31.1
- net GND: now also C29.2; no longer R31.2
- net S3.AIN1: now also C29.1, R38.1; no longer R32.1
- net S3.SWIM_RST: now also R37.2
- net S3.SWIM_RST_IN: now also R37.1
- net S3.T_JTMS: now also R19.1; no longer R19.2
- net S3.T_SWDIO_IN: now also R19.2; no longer R19.1
Other:
- note added: "Not used currently."
- note added: "SWIM dummy circuit."
- moved on the sheet: C18, R19, R21, R29, R30, TP1
