File: pcb/stm32-2inch40.brd (EAGLE design)
At the start: 69.8 x 58.4 mm, 105 parts, among them IC1 CAT24M01WI-GT3, IC2 STM32F103RBT6, IC3 AMIS30663CANG2G, IC4 MAX487-S, Q1 32768Hz, Q2 8MHz, Q3 MMBT2222, SW1 KSS-2EG4430, SW2 KSS-2EG4430, SW3 KSS-2EG4430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

Commit message: Some fixes
Parts:
- added C24: 0.1, rc-master-smd:C0603
- G1: value (none) -> 3V
- JP1: value (none) -> UART
- LCD1: value (none) -> STE2007 (Nokia1202)
- LED1: value (none) -> Green
- LED2: value (none) -> Red
- R16: value 1K -> 2K
- U1: value (none) -> L1117-3.3
- moved R6 7.05 mm to (6.67, 6.99), turned to 180 degrees
- moved R5 5.72 mm to (6.67, 10.2), flipped to the top, turned to 180 degrees
- moved LED1 0.63 mm to (3.17, 10.2)
- moved LED2 0.63 mm to (3.17, 6.99)
Connections:
- net GND: now also C24.2
- net PA0: now also C24.1
Routing:
- net BOOT1: track 32.9 -> 42.2 mm
- net +3V3: track 183.4 -> 190.5 mm
- net N$30: track 6.10 -> 1.68 mm
- net N$13: track 3.93 -> 1.68 mm, vias 1 -> 0
- net PA0: track 53.4 -> 55.5 mm
- net N$3: track 55.6 -> 54.9 mm
- net GND: vias 91 -> 93
