File: pcb/stm32-2inch40-usb-sd-proto.sch (EAGLE design)
At the start: 126 parts, among them IC1 CAT24M01WI-GT3, IC2 STM32F103RBT6, IC4 MAX487-S, K1 ZF112, K2 ZF112, Q1 32768Hz, Q2 8MHz, Q3 MMBT2222, Q4 MMBT2222, Q6 MMBT2222, SW1 KSS-2EG4430, SW2 KSS-2EG4430, SW3 KSS-2EG4430, SW4 KSS-2EG4430, SW5 KSS-2EG4430, U1 L1117-3.3, U2 L1117-3.3, X1 MCV3, X2 MKDSN1,5/2-5,08, X3 MKDSN1,5/6-5,08

Commit message: production ready, small fixes
Parts:
- C10, C11: value 0.1 -> 22pF
- C15, C16: device rc-master-smd:C_0805 -> rc-master-smd:C_0603
- C18: value 47pF -> 0.1
- C19: value 47pF -> 0.1; device rc-master-smd:C_0603 -> rc-master-smd:C_0805
- C20, C27: value 10uF -> 0.1
- C24: value 0.1 -> 10uF; device rc-master-smd:C_0603 -> rc-master-smd:C_0805
- C25: value 0.1 -> 10uF
- C3: value 0.1 -> 47pF
- C4: value 10pF -> 47pF
- C5: value 10pF -> 0.1
- C6, C7: value 22pF -> 0.1
- C8, C9: value 0.1 -> 10pF
- D1: value PESD1CAN -> (none); device protect:PESD1CAN -> semicon-smd-ipc:D-SOD-87
- D2: value (none) -> PESD1CAN; device semicon-smd-ipc:D-SOD-87 -> protect:PESD1CAN
- IC3: value (none) -> MAX487-S; device esp-modules:ESP-12 -> rs232-rs485:MAX487-S
- IC4: value MAX487-S -> (none); device rs232-rs485:MAX487-S -> esp-modules:ESP-12
- L1: value bead -> FB_0603
- L2: value FB_0603 -> bead
- Q1: value 32768Hz -> (none); device crystal:CRSTL3- -> semiconductor:PNP-SOT23
- Q2: value 8MHz -> 32768Hz; device discrete:CRYSTAL-HC49S -> crystal:CRSTL3-
- Q3: value MMBT2222 -> 8MHz; device semiconductor:MMBT2222 -> discrete:CRYSTAL-HC49S
- Q5: value (none) -> MMBT2222; device semiconductor:PNP-SOT23 -> semiconductor:MMBT2222
- R10: value 2.2K -> 4.7K
- R12: value 1K -> 1.5K
- R13: value 2K -> 220
- R14: value 3.9K -> 220
- R15: value 1M -> 10K
- R16: value 2K -> 10K
- R17: value 200 -> 2.2K
- R18: value 200 -> 10K
- R19: value 200 -> 1K
- R20: value 4.7K -> 2K
- R21: value 10 -> 3.9K
- R22: value 2K -> 1M
- R23: value 10K -> 2K
- R24: value 10K -> 200; device rc-master-smd:R_0805 -> rc-master-smd:R_0603
- R25, R26: value 10 -> 200
- R27: value 10 -> 4.7K
- R29: value 10 -> 2K
- R3, R4: value 4.7K -> 10K
- R30, R52: value 10 -> 10K
- R41, R43, R45: value 10K -> 10
- R42: value 1.5K -> 10
- R44, R46: value 560 -> 10
- R48: value 10K -> 560
- R49: value 22 -> 560
- R5, R6: value 220 -> 22
- R50: value 22 -> 10; device rc-master-smd:R_0603 -> rc-master-smd:R_0805
- R53, R54: value 10K -> 1K
- R55, R56: value 1K -> 10K
- R8: value 10K -> 4.7K
- renumbered ESBOOT to SW7, ESRST to SW6, STAMP to STMP1, U$1 to LOGO1
Connections:
- net !LCD_CS: now also R26.2, R27.1; no longer R19.2, R20.1
- net !RESET: now also C6.1, R18.1; no longer C3.1, R11.1
- net !SD_CS: now also R3.1; no longer R43.1
- net !SD_DET: now also R4.1; no longer R45.1
- net +3V3: now also C14.1, C17.1, C20.1, Q1.E, R10.2, R13.1, R18.2, R27.2, R28.2, R30.2, R8.2; no longer C10.1, C8.1, C9.1, Q5.E, R11.2, R20.2, R21.2, R23.2, R3.2, R4.2, R5.1
- net +5V: now also C18.1, C19.1, D1.C, IC3G$2.VCC, R49.2; no longer C14.1, C15.1, D2.C, IC4G$2.VCC, R46.2
- net +5V1: now also C24.1; no longer C27.1
- net BOOT0: now also R15.1; no longer R8.1
- net BOOT1: now also R14.1, R16.1; no longer R6.1, R9.1
- net DE3: now also IC3G$1.DI; no longer IC4G$1.DI
- net ES_3V3: now also C27.1, IC4.3V3, R50.1; no longer C20.1, IC3.3V3, R52.1
- net ES_ADC: now also IC4.ADC; no longer IC3.ADC
- net ES_CHEN: now also IC4.CH_EN, R50.2; no longer IC3.CH_EN, R52.2
- net ES_GND: now also C24.2, IC4.GND, Q5.E, R52.1, R55.1, R56.1; no longer C20.2, IC3.GND, Q4.E, R24.1, R53.1, R54.1
- net ES_GPIO0: now also IC4.GPIO0/!BOOT; no longer IC3.GPIO0/!BOOT
- net ES_GPIO12: now also IC4.GPIO12; no longer IC3.GPIO12
- net ES_GPIO13: now also IC4.GPIO13; no longer IC3.GPIO13
- net ES_GPIO14: now also IC4.GPIO14; no longer IC3.GPIO14
- net ES_GPIO15: now also IC4.GPIO15, R52.2; no longer IC3.GPIO15, R24.2
- net ES_GPIO16: now also IC4.GPIO16; no longer IC3.GPIO16
- net ES_GPIO2: now also IC4.GPIO2; no longer IC3.GPIO2
- net ES_GPIO4: now also IC4.GPIO4; no longer IC3.GPIO4
- net ES_GPIO5: now also IC4.GPIO5; no longer IC3.GPIO5
- net ES_K1: now also R53.1; no longer R55.1
- net ES_K2: now also R54.1; no longer R56.1
- net ES_RST: now also IC4.!RSTB; no longer IC3.!RSTB
- net ES_RXD: now also IC4.RXD; no longer IC3.RXD
- net ES_TXD: now also IC4.TXD; no longer IC3.TXD
- net GND: now also C20.2, D2.3, IC3G$2.GND, Q2.P$1, Q4.E, R16.2, R17.1, R23.1, R47.1, R48.1; no longer C7.2, D1.3, IC4G$2.GND, Q1.P$1, Q3.E, R10.1, R16.1, R41.1, R44.1, R9.2
- net LCD_CLK: now also R25.2; no longer R18.2
- net LCD_DATA: now also R24.2; no longer R17.2
- net N$1: now also Q1.C, R12.2; no longer Q5.C, R42.2
- net N$10: now also R5.1; no longer R49.1
- net N$11: now also R39.1; no longer R33.1
- net N$13: now also R13.2; no longer R5.2
- net N$14: now also R40.1; no longer R34.1
- net N$15: now also R31.1; no longer R25.1
- net N$16: now also R32.1; no longer R26.1
- net N$17: now also R33.1; no longer R27.1
- net N$18: now also R34.1; no longer R28.1
- net N$19: now also R35.1; no longer R29.1
- net N$2: now also D1.A; no longer D2.A
- net N$20: now also R36.1; no longer R30.1
- net N$21: now also R37.1; no longer R31.1
- net N$22: now also R38.1; no longer R32.1
- net N$23: now also R41.1; no longer R35.1
- net N$24: now also R42.1; no longer R36.1
- net N$25: now also R43.1; no longer R37.1
- net N$26: now also R44.1; no longer R38.1
- net N$27: now also R45.1; no longer R39.1
- net N$28: now also R46.1; no longer R40.1
- net N$29: now also Q4.C; no longer Q3.C
- net N$3: now also R15.2, R17.2; no longer R10.2, R8.2
- net N$30: now also R14.2; no longer R6.2
- net N$31: now also R28.1; no longer R21.1
- net N$32: now also Q4.B, R29.1; no longer Q3.B, R22.1
- net N$33: now also R19.1; no longer R12.1
- net N$34: now also R20.1; no longer R13.1
- net N$35: now also R21.1; no longer R14.1
- net N$36: now also R6.1; no longer R50.1
- net N$37: now also Q6.B, R54.2; no longer Q4.B, R53.2
- net N$38: now also Q1.B; no longer Q5.B
- net N$41: now also Q6.C; no longer Q4.C
- net N$42: now also Q5.C; no longer Q6.C
- net N$44: now also D2.1, IC3G$1.A, R49.1; no longer D1.1, IC4G$1.A, R46.1
- net N$46: now also Q5.B, R53.2; no longer Q6.B, R54.2
- net N$6: now also D2.2, IC3G$1.B, R48.2; no longer D1.2, IC4G$1.B, R44.2
- net N$7: now also C5.1, L1.2, R11.2, R3.2, R4.2, R9.2; no longer C17.1, L2.2, R43.2, R45.2, R47.2, R48.2
- net N$8: now also R11.1; no longer R48.1
- net N$9: now also R9.1; no longer R47.1
- net OSC32_IN: now also C8.1, Q2.2; no longer C4.1, Q1.2
- net OSC32_OUT: now also C9.1, Q2.1; no longer C5.1, Q1.1
- net OSC_IN: now also C10.1, Q3.1, R22.2; no longer C6.1, Q2.1, R15.2
- net OSC_OUT: now also C11.1, Q3.2, R22.1; no longer C7.1, Q2.2, R15.1
- net PA0: now also C7.2, R19.2, R20.2, R21.2, R23.2; no longer C24.2, R12.2, R13.2, R14.2, R16.2
- net PA1: now also R26.1; no longer R19.1
- net PA2: now also R24.1; no longer R17.1
- net PA4: now also R25.1; no longer R18.1
- net PB0: now also R45.2; no longer R39.2
- net PB1: now also R46.2; no longer R40.2
- net PB4: now also R29.2; no longer R22.2
- net PC0: now also R39.2; no longer R33.2
- net PC1: now also R40.2; no longer R34.2
- net PC2: now also R41.2; no longer R35.2
- net PC3: now also R42.2; no longer R36.2
- net PC4: now also R43.2; no longer R37.2
- net PC5: now also R44.2; no longer R38.2
- net RXD1: now also R30.1; no longer R23.1
- net RXD3: now also IC3G$1.RO; no longer IC4G$1.RO
- net SCL2: now also R8.1; no longer R3.1
- net SDA2: now also R10.1; no longer R4.1
- net TIM3_CH1: now also R31.2; no longer R25.2
- net TIM3_CH2: now also R32.2; no longer R26.2
- net TIM3_CH3: now also R33.2; no longer R27.2
- net TIM3_CH4: now also R34.2; no longer R28.2
- net TIM4_CH1: now also R35.2; no longer R29.2
- net TIM4_CH2: now also R36.2; no longer R30.2
- net TIM4_CH3: now also R37.2; no longer R31.2
- net TIM4_CH4: now also R38.2; no longer R32.2
- net TXD3: now also IC3G$1.DE, IC3G$1.RE/, R47.2; no longer IC4G$1.DE, IC4G$1.RE/, R41.2
- net USB_DM: now also C3.1, R6.2; no longer C18.1, R50.2
- net USB_DP: now also C4.1, R12.1, R5.2; no longer C19.1, R42.1, R49.2
- net VDDA: now also C15.1, C7.1, L2.2; no longer C11.1, C24.1, L1.2
Other:
- moved on the sheet: C10, C11, C12, C13, C17, C25, C27, C28, C3, C4, C5, C6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

Commit message: change link on silk layer
Parts:
- renumbered STMP1 to STMP
